File: bldc-esc.kicad_pcb (KiCad board)
At the start: 4 copper layers, 0 parts

Commit message: devlog 02
Parts:
- added C101: 100u 63V, Capacitor_SMD:CP_Elec_10x12.5, F.Cu at (30.0, 30.0)
- added C102: 100u 63V, Capacitor_SMD:CP_Elec_10x12.5, F.Cu at (62.0, 30.0)
- added C103: 100u 63V, Capacitor_SMD:CP_Elec_10x12.5, F.Cu at (94.0, 30.0)
- added C104: 100u 63V, Capacitor_SMD:CP_Elec_10x12.5, F.Cu at (126.0, 30.0)
- added C105: 100u 63V, Capacitor_SMD:CP_Elec_10x12.5, F.Cu at (158.0, 30.0)
- added C106: 100u 63V, Capacitor_SMD:CP_Elec_10x12.5, F.Cu at (190.0, 30.0)
- added C107: 100u 63V, Capacitor_SMD:CP_Elec_10x12.5, F.Cu at (222.0, 30.0)
- added C108: 100u 63V, Capacitor_SMD:CP_Elec_10x12.5, F.Cu at (254.0, 30.0)
- added C109: 4.7n 1kV, Capacitor_SMD:C_1206_3216Metric, F.Cu at (286.0, 30.0)
- added C110: 10n 50V, Capacitor_SMD:C_0603_1608Metric, F.Cu at (318.0, 30.0)
- added C111: 10n 50V, Capacitor_SMD:C_0603_1608Metric, F.Cu at (350.0, 30.0)
- added C112: 10n 50V, Capacitor_SMD:C_0603_1608Metric, F.Cu at (382.0, 30.0)
- added C113: 100n 50V, Capacitor_SMD:C_0603_1608Metric, F.Cu at (414.0, 30.0)
- added C114: 100n 50V, Capacitor_SMD:C_0603_1608Metric, F.Cu at (446.0, 30.0)
- added C115: 100u 63V, Capacitor_SMD:CP_Elec_10x12.5, F.Cu at (478.0, 30.0)
- added C116: 100u 63V, Capacitor_SMD:CP_Elec_10x12.5, F.Cu at (510.0, 30.0)
- added C201: 22u 63V, Capacitor_THT:CP_Radial_D6.3mm_P2.50mm, F.Cu at (542.0, 30.0)
- added C202: 100n 100V, Capacitor_SMD:C_0603_1608Metric, F.Cu at (574.0, 30.0)
- added C203: 47n 100V, Capacitor_SMD:C_0805_2012Metric, F.Cu at (30.0, 62.0)
- added C204: 1u 50V, Capacitor_SMD:C_1206_3216Metric, F.Cu at (62.0, 62.0)
- added C205: 1u 25V, Capacitor_SMD:C_0805_2012Metric, F.Cu at (94.0, 62.0)
- added C206: 1u 16V, Capacitor_SMD:C_0603_1608Metric, F.Cu at (126.0, 62.0)
- added C207: 100n 50V, Capacitor_SMD:C_0603_1608Metric, F.Cu at (158.0, 62.0)
- added C210: 1u 100V, Capacitor_SMD:C_1206_3216Metric, F.Cu at (190.0, 62.0)
- added C211: 1u 100V, Capacitor_SMD:C_1206_3216Metric, F.Cu at (222.0, 62.0)
- added C212: 100n 50V, Capacitor_SMD:C_0603_1608Metric, F.Cu at (254.0, 62.0)
- added C213: 1n 50V, Capacitor_SMD:C_0603_1608Metric, F.Cu at (286.0, 62.0)
- added C214: 1n 50V, Capacitor_SMD:C_0603_1608Metric, F.Cu at (318.0, 62.0)
- added C215: 1n 100V, Capacitor_SMD:C_0805_2012Metric, F.Cu at (350.0, 62.0)
- added C230: 1u 100V, Capacitor_SMD:C_1206_3216Metric, F.Cu at (382.0, 62.0)
- added C231: 1u 100V, Capacitor_SMD:C_1206_3216Metric, F.Cu at (414.0, 62.0)
- added C232: 100n 50V, Capacitor_SMD:C_0603_1608Metric, F.Cu at (446.0, 62.0)
- added C233: 1n 50V, Capacitor_SMD:C_0603_1608Metric, F.Cu at (478.0, 62.0)
- added C234: 1n 50V, Capacitor_SMD:C_0603_1608Metric, F.Cu at (510.0, 62.0)
- added C235: 1n 100V, Capacitor_SMD:C_0805_2012Metric, F.Cu at (542.0, 62.0)
- added C250: 1u 100V, Capacitor_SMD:C_1206_3216Metric, F.Cu at (574.0, 62.0)
- added C251: 1u 100V, Capacitor_SMD:C_1206_3216Metric, F.Cu at (30.0, 94.0)
- added C252: 100n 50V, Capacitor_SMD:C_0603_1608Metric, F.Cu at (62.0, 94.0)
- added C253: 1n 50V, Capacitor_SMD:C_0603_1608Metric, F.Cu at (94.0, 94.0)
- added C254: 1n 50V, Capacitor_SMD:C_0603_1608Metric, F.Cu at (126.0, 94.0)
- added C255: 1n 100V, Capacitor_SMD:C_0805_2012Metric, F.Cu at (158.0, 94.0)
- added C301: 1n 50V, Capacitor_SMD:C_0603_1608Metric, F.Cu at (190.0, 94.0)
- added C302: 100n 50V, Capacitor_SMD:C_0603_1608Metric, F.Cu at (222.0, 94.0)
- added C303: 1n 50V, Capacitor_SMD:C_0603_1608Metric, F.Cu at (254.0, 94.0)
- added C304: 100n 50V, Capacitor_SMD:C_0603_1608Metric, F.Cu at (286.0, 94.0)
- added C305: 1u 16V, Capacitor_SMD:C_0603_1608Metric, F.Cu at (318.0, 94.0)
- added C306: 100n 50V, Capacitor_SMD:C_0603_1608Metric, F.Cu at (350.0, 94.0)
- added C307: 100n 50V, Capacitor_SMD:C_0603_1608Metric, F.Cu at (382.0, 94.0)
- added C308: 100p 50V, Capacitor_SMD:C_0603_1608Metric, F.Cu at (414.0, 94.0)
- added C309: 100n 50V, Capacitor_SMD:C_0603_1608Metric, F.Cu at (446.0, 94.0)
- added C310: 10n 50V, Capacitor_SMD:C_0603_1608Metric, F.Cu at (478.0, 94.0)
- added C311: 100n 50V, Capacitor_SMD:C_0603_1608Metric, F.Cu at (510.0, 94.0)
- added C401: 2.2u 100V, Capacitor_SMD:C_1206_3216Metric, F.Cu at (542.0, 94.0)
- added C402: 2.2u 100V, Capacitor_SMD:C_1206_3216Metric, F.Cu at (574.0, 94.0)
- added C403: 2.2n 50V, Capacitor_SMD:C_0603_1608Metric, F.Cu at (30.0, 126.0)
- added C404: 22u 25V, Capacitor_SMD:C_1210_3225Metric, F.Cu at (62.0, 126.0)
- added C405: 22u 25V, Capacitor_SMD:C_1210_3225Metric, F.Cu at (94.0, 126.0)
- added C406: 2.2n 50V, Capacitor_SMD:C_0603_1608Metric, F.Cu at (126.0, 126.0)
- added C407: 82p 50V, Capacitor_SMD:C_0603_1608Metric, F.Cu at (158.0, 126.0)
- added C408: 1u 16V, Capacitor_SMD:C_0603_1608Metric, F.Cu at (190.0, 126.0)
- added C409: 1u 16V, Capacitor_SMD:C_0603_1608Metric, F.Cu at (222.0, 126.0)
- added C410: 4.7u 10V, Capacitor_SMD:C_0805_2012Metric, F.Cu at (254.0, 126.0)
- added C411: 1u 16V, Capacitor_SMD:C_0603_1608Metric, F.Cu at (286.0, 126.0)
- added C412: 4.7u 10V, Capacitor_SMD:C_0805_2012Metric, F.Cu at (318.0, 126.0)
- added C413: 100n 50V, Capacitor_SMD:C_0603_1608Metric, F.Cu at (350.0, 126.0)
- added C501: 100n 50V, Capacitor_SMD:C_0603_1608Metric, F.Cu at (382.0, 126.0)
- added C502: 100n 50V, Capacitor_SMD:C_0603_1608Metric, F.Cu at (414.0, 126.0)
- added C503: 100n 50V, Capacitor_SMD:C_0603_1608Metric, F.Cu at (446.0, 126.0)
- added C504: 100n 50V, Capacitor_SMD:C_0603_1608Metric, F.Cu at (478.0, 126.0)
- added C505: 100n 50V, Capacitor_SMD:C_0603_1608Metric, F.Cu at (510.0, 126.0)
- added C506: 4.7u 10V, Capacitor_SMD:C_0805_2012Metric, F.Cu at (542.0, 126.0)
- added C507: 4.7u 10V, Capacitor_SMD:C_0805_2012Metric, F.Cu at (574.0, 126.0)
- added C508: 100n 50V, Capacitor_SMD:C_0603_1608Metric, F.Cu at (30.0, 158.0)
- added C509: 100n 50V, Capacitor_SMD:C_0603_1608Metric, F.Cu at (62.0, 158.0)
- added C510: 1u 16V, Capacitor_SMD:C_0603_1608Metric, F.Cu at (94.0, 158.0)
- added C511: 100n 50V, Capacitor_SMD:C_0603_1608Metric, F.Cu at (126.0, 158.0)
- added C512: 100n 50V, Capacitor_SMD:C_0603_1608Metric, F.Cu at (158.0, 158.0)
- added C513: 27p 50V, Capacitor_SMD:C_0603_1608Metric, F.Cu at (190.0, 158.0)
- added C514: 27p 50V, Capacitor_SMD:C_0603_1608Metric, F.Cu at (222.0, 158.0)
- added C515: 100n 50V, Capacitor_SMD:C_0603_1608Metric, F.Cu at (254.0, 158.0)
- added C516: 100n 50V, Capacitor_SMD:C_0603_1608Metric, F.Cu at (286.0, 158.0)
- added C517: 100n 50V, Capacitor_SMD:C_0603_1608Metric, F.Cu at (318.0, 158.0)
- added C601: 100n 50V, Capacitor_SMD:C_0603_1608Metric, F.Cu at (350.0, 158.0)
- added C602: 1u 16V, Capacitor_SMD:C_0603_1608Metric, F.Cu at (382.0, 158.0)
- added C603: 100n 50V, Capacitor_SMD:C_0603_1608Metric, F.Cu at (414.0, 158.0)
- added C604: 1u 16V, Capacitor_SMD:C_0603_1608Metric, F.Cu at (446.0, 158.0)
- added C605: 100n 50V, Capacitor_SMD:C_0603_1608Metric, F.Cu at (478.0, 158.0)
- added C606: 100n 50V, Capacitor_SMD:C_0603_1608Metric, F.Cu at (510.0, 158.0)
- added C610: 100p 50V, Capacitor_SMD:C_0603_1608Metric, F.Cu at (542.0, 158.0)
- added C611: 100p 50V, Capacitor_SMD:C_0603_1608Metric, F.Cu at (574.0, 158.0)
- added C612: 100p 50V, Capacitor_SMD:C_0603_1608Metric, F.Cu at (30.0, 190.0)
- added C613: 100p 50V, Capacitor_SMD:C_0603_1608Metric, F.Cu at (62.0, 190.0)
- added C614: 100p 50V, Capacitor_SMD:C_0603_1608Metric, F.Cu at (94.0, 190.0)
- added C615: 100p 50V, Capacitor_SMD:C_0603_1608Metric, F.Cu at (126.0, 190.0)
- added C701: 100n 50V, Capacitor_SMD:C_0603_1608Metric, F.Cu at (158.0, 190.0)
- added C702: 10n 50V, Capacitor_SMD:C_0603_1608Metric, F.Cu at (190.0, 190.0)
- added C703: 100n 50V, Capacitor_SMD:C_0603_1608Metric, F.Cu at (222.0, 190.0)
- added C704: 100n 50V, Capacitor_SMD:C_0603_1608Metric, F.Cu at (254.0, 190.0)
- added C705: 10n 50V, Capacitor_SMD:C_0603_1608Metric, F.Cu at (286.0, 190.0)
- added C711: 100n 50V, Capacitor_SMD:C_0603_1608Metric, F.Cu at (318.0, 190.0)
- added C712: 100n 50V, Capacitor_SMD:C_0603_1608Metric, F.Cu at (350.0, 190.0)
- added C713: 100n 50V, Capacitor_SMD:C_0603_1608Metric, F.Cu at (382.0, 190.0)
- added C714: 100n 50V, Capacitor_SMD:C_0603_1608Metric, F.Cu at (414.0, 190.0)
- added C715: 100n 50V, Capacitor_SMD:C_0603_1608Metric, F.Cu at (446.0, 190.0)
- added C716: 100n 50V, Capacitor_SMD:C_0603_1608Metric, F.Cu at (478.0, 190.0)
- added C717: 100n 50V, Capacitor_SMD:C_0603_1608Metric, F.Cu at (510.0, 190.0)
- added C718: 100n 50V, Capacitor_SMD:C_0603_1608Metric, F.Cu at (542.0, 190.0)
- added C719: 100n 50V, Capacitor_SMD:C_0603_1608Metric, F.Cu at (574.0, 190.0)
- added C720: 100n 50V, Capacitor_SMD:C_0603_1608Metric, F.Cu at (30.0, 222.0)
- added C801: 220p 50V, Capacitor_SMD:C_0603_1608Metric, F.Cu at (62.0, 222.0)
- added C802: 1n 50V, Capacitor_SMD:C_0603_1608Metric, F.Cu at (94.0, 222.0)
- added C811: 220p 50V, Capacitor_SMD:C_0603_1608Metric, F.Cu at (126.0, 222.0)
- added C812: 1n 50V, Capacitor_SMD:C_0603_1608Metric, F.Cu at (158.0, 222.0)
- added C821: 220p 50V, Capacitor_SMD:C_0603_1608Metric, F.Cu at (190.0, 222.0)
- added C822: 1n 50V, Capacitor_SMD:C_0603_1608Metric, F.Cu at (222.0, 222.0)
- added C831: 220p 50V, Capacitor_SMD:C_0603_1608Metric, F.Cu at (254.0, 222.0)
- added C832: 1n 50V, Capacitor_SMD:C_0603_1608Metric, F.Cu at (286.0, 222.0)
- added C840: 100n 50V, Capacitor_SMD:C_0603_1608Metric, F.Cu at (318.0, 222.0)
- added C845: 100n 50V, Capacitor_SMD:C_0603_1608Metric, F.Cu at (350.0, 222.0)
- added C850: 10n 50V, Capacitor_SMD:C_0603_1608Metric, F.Cu at (382.0, 222.0)
- added C855: 10n 50V, Capacitor_SMD:C_0603_1608Metric, F.Cu at (414.0, 222.0)
- added C865: 1n 50V, Capacitor_SMD:C_0603_1608Metric, F.Cu at (446.0, 222.0)
- added C868: 1n 50V, Capacitor_SMD:C_0603_1608Metric, F.Cu at (478.0, 222.0)
- added C871: 1n 50V, Capacitor_SMD:C_0603_1608Metric, F.Cu at (510.0, 222.0)
- added C880: 10n 50V, Capacitor_SMD:C_0603_1608Metric, F.Cu at (542.0, 222.0)
- added C883: 10n 50V, Capacitor_SMD:C_0603_1608Metric, F.Cu at (574.0, 222.0)
- added C886: 10n 50V, Capacitor_SMD:C_0603_1608Metric, F.Cu at (30.0, 254.0)
- added C889: 10n 50V, Capacitor_SMD:C_0603_1608Metric, F.Cu at (62.0, 254.0)
- added C899: 10n 50V, Capacitor_SMD:C_0603_1608Metric, F.Cu at (94.0, 254.0)
- added D101: SMCJ30A, Diode_SMD:D_SMC, F.Cu at (126.0, 254.0)
- added D301: STPS5H100B, Diode_SMD:D_SMC, F.Cu at (158.0, 254.0)
- added D302: BAT54H, Diode_SMD:D_SOD-123F, F.Cu at (190.0, 254.0)
- added D303: BAT54H, Diode_SMD:D_SOD-123F, F.Cu at (222.0, 254.0)
- added D501: PMEG2010ER, Diode_SMD:Nexperia_CFP3_SOD-123W, F.Cu at (254.0, 254.0)
- added D511: STATUS, LED_SMD:LED_0603_1608Metric, F.Cu at (286.0, 254.0)
- added D512: COMM, LED_SMD:LED_0603_1608Metric, F.Cu at (318.0, 254.0)
- added D513: POWER, LED_SMD:LED_0603_1608Metric, F.Cu at (350.0, 254.0)
- added D610: PESD5V0S1BA, Diode_SMD:D_SOD-323, F.Cu at (382.0, 254.0)
- added D611: PESD5V0S1BA, Diode_SMD:D_SOD-323, F.Cu at (414.0, 254.0)
- added D612: PESD5V0S1BA, Diode_SMD:D_SOD-323, F.Cu at (446.0, 254.0)
- added D613: PESD5V0S1BA, Diode_SMD:D_SOD-323, F.Cu at (478.0, 254.0)
- added D614: PESD5V0S1BA, Diode_SMD:D_SOD-323, F.Cu at (510.0, 254.0)
- added D615: PESD5V0S1BA, Diode_SMD:D_SOD-323, F.Cu at (542.0, 254.0)
- added D701: BAT54H, Diode_SMD:D_SOD-123F, F.Cu at (574.0, 254.0)
- added D702: BAT54H, Diode_SMD:D_SOD-123F, F.Cu at (30.0, 286.0)
- added D703: PESD2CANFD24V-T, Package_TO_SOT_SMD:SOT-23, F.Cu at (62.0, 286.0)
- added D801: BAT54S, Package_TO_SOT_SMD:SOT-23, F.Cu at (94.0, 286.0)
- added D811: BAT54S, Package_TO_SOT_SMD:SOT-23, F.Cu at (126.0, 286.0)
- added D821: BAT54S, Package_TO_SOT_SMD:SOT-23, F.Cu at (158.0, 286.0)
- added D831: BAT54S, Package_TO_SOT_SMD:SOT-23, F.Cu at (190.0, 286.0)
- added D850: BAT54S, Package_TO_SOT_SMD:SOT-23, F.Cu at (222.0, 286.0)
- added D855: BAT54S, Package_TO_SOT_SMD:SOT-23, F.Cu at (254.0, 286.0)
- added D865: PESD5V0S1BA, Diode_SMD:D_SOD-323, F.Cu at (286.0, 286.0)
- added D868: PESD5V0S1BA, Diode_SMD:D_SOD-323, F.Cu at (318.0, 286.0)
- added D871: PESD5V0S1BA, Diode_SMD:D_SOD-323, F.Cu at (350.0, 286.0)
- added D886: BAT54S, Package_TO_SOT_SMD:SOT-23, F.Cu at (382.0, 286.0)
- added D889: BAT54S, Package_TO_SOT_SMD:SOT-23, F.Cu at (414.0, 286.0)
- added F401: 0.5A / 6V, Fuse:Fuse_1206_3216Metric, F.Cu at (446.0, 286.0)
- added FB501: 600R @ 100MHz, Inductor_SMD:L_0603_1608Metric, F.Cu at (478.0, 286.0)
- added J101: XT60PW-M, Connector_AMASS:AMASS_XT60PW-M_1x02_P7.20mm_Horizontal, F.Cu at (510.0, 286.0)
- added J102: MT60 / 12AWG pigtail, bldc-esc:MT60_Pigtail_12AWG, F.Cu at (542.0, 286.0)
- added J103: CHASSIS, Connector_PinHeader_2.54mm:PinHeader_1x02_P2.54mm_Vertical, F.Cu at (574.0, 286.0)
- added J301: DUMP RESISTOR, TerminalBlock_Phoenix:TerminalBlock_Phoenix_MKDS-3-2-5.08_1x02_P5.08mm_Horizontal, F.Cu at (30.0, 318.0)
- added J401: USB4105-GF-A, Connector_USB:USB_C_Receptacle_GCT_USB4105-xx-A_16P_TopMnt_Horizontal, F.Cu at (62.0, 318.0)
- added J501: SWD, Connector_PinHeader_1.27mm:PinHeader_2x05_P1.27mm_Vertical_SMD, F.Cu at (94.0, 318.0)
- added J601: HALL, Connector_JST:JST_GH_BM05B-GHS-TBT_1x05-1MP_P1.25mm_Vertical, F.Cu at (126.0, 318.0)
- added J602: ENCODER, Connector_JST:JST_GH_BM05B-GHS-TBT_1x05-1MP_P1.25mm_Vertical, F.Cu at (158.0, 318.0)
- added J701: CAN, Connector_JST:JST_GH_BM03B-GHS-TBT_1x03-1MP_P1.25mm_Vertical, F.Cu at (190.0, 318.0)
- added J702: UART / 3V3, Connector_JST:JST_GH_BM04B-GHS-TBT_1x04-1MP_P1.25mm_Vertical, F.Cu at (222.0, 318.0)
- added J703: HW ENABLE, Connector_PinHeader_2.54mm:PinHeader_1x02_P2.54mm_Vertical, F.Cu at (254.0, 318.0)
- added J801: THROTTLE_ADC, Connector_JST:JST_GH_BM03B-GHS-TBT_1x03-1MP_P1.25mm_Vertical, F.Cu at (286.0, 318.0)
- added J802: AUX_ANALOG_ADC, Connector_JST:JST_GH_BM03B-GHS-TBT_1x03-1MP_P1.25mm_Vertical, F.Cu at (318.0, 318.0)
- added J803: RC PWM, Connector_JST:JST_GH_BM03B-GHS-TBT_1x03-1MP_P1.25mm_Vertical, F.Cu at (350.0, 318.0)
- added J804: BRAKE / DIR, Connector_JST:JST_GH_BM03B-GHS-TBT_1x03-1MP_P1.25mm_Vertical, F.Cu at (382.0, 318.0)
- added J805: NTC_MOTOR, Connector_JST:JST_GH_BM02B-GHS-TBT_1x02-1MP_P1.25mm_Vertical, F.Cu at (414.0, 318.0)
- added J806: NTC_DUMP, Connector_JST:JST_GH_BM02B-GHS-TBT_1x02-1MP_P1.25mm_Vertical, F.Cu at (446.0, 318.0)
- added JP501: BOOT0, Connector_PinHeader_2.54mm:PinHeader_1x02_P2.54mm_Vertical, F.Cu at (478.0, 318.0)
- added JP701: CAN TERM, Connector_PinHeader_2.54mm:PinHeader_1x02_P2.54mm_Vertical, F.Cu at (510.0, 318.0)
- added JP704: RUN 1-2 / SERVICE 2-3, Connector_PinHeader_2.54mm:PinHeader_1x03_P2.54mm_Vertical, F.Cu at (542.0, 318.0)
- added L401: 68uH / Isat>=1.8A, Inductor_SMD:L_Coilcraft_MSS1246T-XXX, F.Cu at (574.0, 318.0)
- added Q201: ISC011N06LM5, Package_SON:Infineon_PG-TDSON-8_6.15x5.15mm, F.Cu at (30.0, 350.0)
- added Q202: ISC011N06LM5, Package_SON:Infineon_PG-TDSON-8_6.15x5.15mm, F.Cu at (62.0, 350.0)
- added Q203: ISC011N06LM5, Package_SON:Infineon_PG-TDSON-8_6.15x5.15mm, F.Cu at (94.0, 350.0)
- added Q204: ISC011N06LM5, Package_SON:Infineon_PG-TDSON-8_6.15x5.15mm, F.Cu at (126.0, 350.0)
- added Q205: ISC011N06LM5, Package_SON:Infineon_PG-TDSON-8_6.15x5.15mm, F.Cu at (158.0, 350.0)
- added Q206: ISC011N06LM5, Package_SON:Infineon_PG-TDSON-8_6.15x5.15mm, F.Cu at (190.0, 350.0)
- added Q301: ISC011N06LM5, Package_SON:Infineon_PG-TDSON-8_6.15x5.15mm, F.Cu at (222.0, 350.0)
- added Q302: 2N7002, Package_TO_SOT_SMD:SOT-23, F.Cu at (254.0, 350.0)
- added R101: 10k, Resistor_SMD:R_1206_3216Metric, F.Cu at (286.0, 350.0)
- added R102: 1M, Resistor_SMD:R_0603_1608Metric, F.Cu at (318.0, 350.0)
- added R103: 0, Resistor_SMD:R_0603_1608Metric, F.Cu at (350.0, 350.0)
- added R110: 10k 0.1%, Resistor_SMD:R_0603_1608Metric, F.Cu at (382.0, 350.0)
- added R111: 49.9k 0.1%, Resistor_SMD:R_0603_1608Metric, F.Cu at (414.0, 350.0)
- added R112: 49.9k 0.1%, Resistor_SMD:R_0603_1608Metric, F.Cu at (446.0, 350.0)
- added R113: 10k 0.1%, Resistor_SMD:R_0603_1608Metric, F.Cu at (478.0, 350.0)
- added R114: 10k 0.1%, Resistor_SMD:R_0603_1608Metric, F.Cu at (510.0, 350.0)
- added R115: 11k 0.1%, Resistor_SMD:R_0603_1608Metric, F.Cu at (542.0, 350.0)
- added R116: 4.7k, Resistor_SMD:R_0603_1608Metric, F.Cu at (574.0, 350.0)
- added R117: 10k, Resistor_SMD:R_0603_1608Metric, F.Cu at (30.0, 382.0)
- added R201: 2.2, Resistor_SMD:R_0805_2012Metric, F.Cu at (62.0, 382.0)
- added R202: 4.7k, Resistor_SMD:R_0603_1608Metric, F.Cu at (94.0, 382.0)
- added R203: 10k, Resistor_SMD:R_0603_1608Metric, F.Cu at (126.0, 382.0)
- added R204: 100k, Resistor_SMD:R_0603_1608Metric, F.Cu at (158.0, 382.0)
- added R205: 10k, Resistor_SMD:R_0603_1608Metric, F.Cu at (190.0, 382.0)
- added R210: 3.3, Resistor_SMD:R_0603_1608Metric, F.Cu at (222.0, 382.0)
- added R211: 47k, Resistor_SMD:R_0603_1608Metric, F.Cu at (254.0, 382.0)
- added R212: 3.3, Resistor_SMD:R_0603_1608Metric, F.Cu at (286.0, 382.0)
- added R213: 47k, Resistor_SMD:R_0603_1608Metric, F.Cu at (318.0, 382.0)
- added R214: 1m 1% 8W, bldc-esc:CSS4J_4026, F.Cu at (350.0, 382.0)
- added R215: 100, Resistor_SMD:R_0603_1608Metric, F.Cu at (382.0, 382.0)
- added R216: 1k, Resistor_SMD:R_0603_1608Metric, F.Cu at (414.0, 382.0)
- added R217: 10, Resistor_SMD:R_0805_2012Metric, F.Cu at (446.0, 382.0)
- added R230: 3.3, Resistor_SMD:R_0603_1608Metric, F.Cu at (478.0, 382.0)
- added R231: 47k, Resistor_SMD:R_0603_1608Metric, F.Cu at (510.0, 382.0)
- added R232: 3.3, Resistor_SMD:R_0603_1608Metric, F.Cu at (542.0, 382.0)
- added R233: 47k, Resistor_SMD:R_0603_1608Metric, F.Cu at (574.0, 382.0)
- added R234: 1m 1% 8W, bldc-esc:CSS4J_4026, F.Cu at (30.0, 414.0)
- added R235: 100, Resistor_SMD:R_0603_1608Metric, F.Cu at (62.0, 414.0)
- added R236: 1k, Resistor_SMD:R_0603_1608Metric, F.Cu at (94.0, 414.0)
- added R237: 10, Resistor_SMD:R_0805_2012Metric, F.Cu at (126.0, 414.0)
- added R250: 3.3, Resistor_SMD:R_0603_1608Metric, F.Cu at (158.0, 414.0)
- added R251: 47k, Resistor_SMD:R_0603_1608Metric, F.Cu at (190.0, 414.0)
- added R252: 3.3, Resistor_SMD:R_0603_1608Metric, F.Cu at (222.0, 414.0)
- added R253: 47k, Resistor_SMD:R_0603_1608Metric, F.Cu at (254.0, 414.0)
- added R254: 1m 1% 8W, bldc-esc:CSS4J_4026, F.Cu at (286.0, 414.0)
- added R255: 100, Resistor_SMD:R_0603_1608Metric, F.Cu at (318.0, 414.0)
- added R256: 1k, Resistor_SMD:R_0603_1608Metric, F.Cu at (350.0, 414.0)
- added R257: 10, Resistor_SMD:R_0805_2012Metric, F.Cu at (382.0, 414.0)
- added R301: 100k 0.1%, Resistor_SMD:R_0603_1608Metric, F.Cu at (414.0, 414.0)
- added R302: 100k 0.1%, Resistor_SMD:R_0603_1608Metric, F.Cu at (446.0, 414.0)
- added R303: 8.45k 0.1%, Resistor_SMD:R_0603_1608Metric, F.Cu at (478.0, 414.0)
- added R304: 10k 0.1%, Resistor_SMD:R_0603_1608Metric, F.Cu at (510.0, 414.0)
- added R305: 2.49M, Resistor_SMD:R_0603_1608Metric, F.Cu at (542.0, 414.0)
- added R306: 4.7k, Resistor_SMD:R_0603_1608Metric, F.Cu at (574.0, 414.0)
- added R307: 2.2, Resistor_SMD:R_0603_1608Metric, F.Cu at (30.0, 446.0)
- added R308: 1, Resistor_SMD:R_0603_1608Metric, F.Cu at (62.0, 446.0)
- added R309: 47k, Resistor_SMD:R_0603_1608Metric, F.Cu at (94.0, 446.0)
- added R310: 3m / 3W, Resistor_SMD:R_2512_6332Metric, F.Cu at (126.0, 446.0)
- added R311: 10k, Resistor_SMD:R_0603_1608Metric, F.Cu at (158.0, 446.0)
- added R312: 10k, Resistor_SMD:R_0603_1608Metric, F.Cu at (190.0, 446.0)
- added R313: 10k, Resistor_SMD:R_0603_1608Metric, F.Cu at (222.0, 446.0)
- added R314: 100k, Resistor_SMD:R_0603_1608Metric, F.Cu at (254.0, 446.0)
- added R315: 100k, Resistor_SMD:R_0603_1608Metric, F.Cu at (286.0, 446.0)
- added R316: 100k, Resistor_SMD:R_0603_1608Metric, F.Cu at (318.0, 446.0)
- added R317: 100k, Resistor_SMD:R_0603_1608Metric, F.Cu at (350.0, 446.0)
- added R318: 100k, Resistor_SMD:R_0603_1608Metric, F.Cu at (382.0, 446.0)
- added R319: 100k, Resistor_SMD:R_0603_1608Metric, F.Cu at (414.0, 446.0)
- added R401: 300k, Resistor_SMD:R_0603_1608Metric, F.Cu at (446.0, 446.0)
- added R402: 100k, Resistor_SMD:R_0603_1608Metric, F.Cu at (478.0, 446.0)
- added R403: 42.2k, Resistor_SMD:R_0603_1608Metric, F.Cu at (510.0, 446.0)
- added R404: 324k 0.1%, Resistor_SMD:R_0603_1608Metric, F.Cu at (542.0, 446.0)
- added R405: 100k 0.1%, Resistor_SMD:R_0603_1608Metric, F.Cu at (574.0, 446.0)
- added R406: 301k, Resistor_SMD:R_0603_1608Metric, F.Cu at (30.0, 478.0)
- added R407: 10k, Resistor_SMD:R_0603_1608Metric, F.Cu at (62.0, 478.0)
- added R408: 300k, Resistor_SMD:R_0603_1608Metric, F.Cu at (94.0, 478.0)
- added R409: 100k, Resistor_SMD:R_0603_1608Metric, F.Cu at (126.0, 478.0)
- added R410: 10k, Resistor_SMD:R_0603_1608Metric, F.Cu at (158.0, 478.0)
- added R411: 5.1k, Resistor_SMD:R_0603_1608Metric, F.Cu at (190.0, 478.0)
- added R412: 5.1k, Resistor_SMD:R_0603_1608Metric, F.Cu at (222.0, 478.0)
- added R413: 22, Resistor_SMD:R_0603_1608Metric, F.Cu at (254.0, 478.0)
- added R414: 22, Resistor_SMD:R_0603_1608Metric, F.Cu at (286.0, 478.0)
- added R415: 100k, Resistor_SMD:R_0603_1608Metric, F.Cu at (318.0, 478.0)
- added R416: 150k, Resistor_SMD:R_0603_1608Metric, F.Cu at (350.0, 478.0)
- added R501: 1k, Resistor_SMD:R_0603_1608Metric, F.Cu at (382.0, 478.0)
- added R502: 0, Resistor_SMD:R_0603_1608Metric, F.Cu at (414.0, 478.0)
- added R503: 100k, Resistor_SMD:R_0603_1608Metric, F.Cu at (446.0, 478.0)
- added R504: 10k, Resistor_SMD:R_0603_1608Metric, F.Cu at (478.0, 478.0)
- added R505: 10k, Resistor_SMD:R_0603_1608Metric, F.Cu at (510.0, 478.0)
- added R506: 4.7k, Resistor_SMD:R_0603_1608Metric, F.Cu at (542.0, 478.0)
- added R507: 4.7k, Resistor_SMD:R_0603_1608Metric, F.Cu at (574.0, 478.0)
- added R508: 10k, Resistor_SMD:R_0603_1608Metric, F.Cu at (30.0, 510.0)
- added R511: 1k, Resistor_SMD:R_0603_1608Metric, F.Cu at (62.0, 510.0)
- added R512: 1k, Resistor_SMD:R_0603_1608Metric, F.Cu at (94.0, 510.0)
- added R513: 1k, Resistor_SMD:R_0603_1608Metric, F.Cu at (126.0, 510.0)
- added R601: 200k, Resistor_SMD:R_0603_1608Metric, F.Cu at (158.0, 510.0)
- added R602: 100k, Resistor_SMD:R_0603_1608Metric, F.Cu at (190.0, 510.0)
- added R603: 10k, Resistor_SMD:R_0603_1608Metric, F.Cu at (222.0, 510.0)
- added R605: 200k, Resistor_SMD:R_0603_1608Metric, F.Cu at (254.0, 510.0)
- added R606: 100k, Resistor_SMD:R_0603_1608Metric, F.Cu at (286.0, 510.0)
- added R607: 10k, Resistor_SMD:R_0603_1608Metric, F.Cu at (318.0, 510.0)
- added R620: 1k, Resistor_SMD:R_0603_1608Metric, F.Cu at (350.0, 510.0)
- added R621: 10k, Resistor_SMD:R_0603_1608Metric, F.Cu at (382.0, 510.0)
- added R623: 1k, Resistor_SMD:R_0603_1608Metric, F.Cu at (414.0, 510.0)
- added R624: 10k, Resistor_SMD:R_0603_1608Metric, F.Cu at (446.0, 510.0)
- added R626: 1k, Resistor_SMD:R_0603_1608Metric, F.Cu at (478.0, 510.0)
- added R627: 10k, Resistor_SMD:R_0603_1608Metric, F.Cu at (510.0, 510.0)
- added R632: 1k, Resistor_SMD:R_0603_1608Metric, F.Cu at (542.0, 510.0)
- added R633: 10k, Resistor_SMD:R_0603_1608Metric, F.Cu at (574.0, 510.0)
- added R635: 1k, Resistor_SMD:R_0603_1608Metric, F.Cu at (30.0, 542.0)
- added R636: 10k, Resistor_SMD:R_0603_1608Metric, F.Cu at (62.0, 542.0)
- added R638: 1k, Resistor_SMD:R_0603_1608Metric, F.Cu at (94.0, 542.0)
- added R639: 10k, Resistor_SMD:R_0603_1608Metric, F.Cu at (126.0, 542.0)
- added R701: 10k, Resistor_SMD:R_0603_1608Metric, F.Cu at (158.0, 542.0)
- added R702: 10k, Resistor_SMD:R_0603_1608Metric, F.Cu at (190.0, 542.0)
- added R703: 10k, Resistor_SMD:R_0603_1608Metric, F.Cu at (222.0, 542.0)
- added R704: 100k, Resistor_SMD:R_0603_1608Metric, F.Cu at (254.0, 542.0)
- added R705: 100k, Resistor_SMD:R_0603_1608Metric, F.Cu at (286.0, 542.0)
- added R706: 10k, Resistor_SMD:R_0603_1608Metric, F.Cu at (318.0, 542.0)
- added R710: 10k, Resistor_SMD:R_0603_1608Metric, F.Cu at (350.0, 542.0)
- added R711: 10k, Resistor_SMD:R_0603_1608Metric, F.Cu at (382.0, 542.0)
- added R712: 10k, Resistor_SMD:R_0603_1608Metric, F.Cu at (414.0, 542.0)
- added R713: 10k, Resistor_SMD:R_0603_1608Metric, F.Cu at (446.0, 542.0)
- added R714: 10k, Resistor_SMD:R_0603_1608Metric, F.Cu at (478.0, 542.0)
- added R715: 10k, Resistor_SMD:R_0603_1608Metric, F.Cu at (510.0, 542.0)
- added R716: 100k, Resistor_SMD:R_0603_1608Metric, F.Cu at (542.0, 542.0)
- added R717: 10k, Resistor_SMD:R_0603_1608Metric, F.Cu at (574.0, 542.0)
- added R718: 10k, Resistor_SMD:R_0603_1608Metric, F.Cu at (30.0, 574.0)
- added R719: 120, Resistor_SMD:R_0805_2012Metric, F.Cu at (62.0, 574.0)
- added R720: 10k, Resistor_SMD:R_0603_1608Metric, F.Cu at (94.0, 574.0)
- added R721: 1k, Resistor_SMD:R_0603_1608Metric, F.Cu at (126.0, 574.0)
- added R722: 10k, Resistor_SMD:R_0603_1608Metric, F.Cu at (158.0, 574.0)
- added R801: 100k 0.1%, Resistor_SMD:R_0603_1608Metric, F.Cu at (190.0, 574.0)
- added R802: 100k 0.1%, Resistor_SMD:R_0603_1608Metric, F.Cu at (222.0, 574.0)
- added R803: 10k 0.1%, Resistor_SMD:R_0603_1608Metric, F.Cu at (254.0, 574.0)
- added R804: 100, Resistor_SMD:R_0603_1608Metric, F.Cu at (286.0, 574.0)
- added R811: 100k 0.1%, Resistor_SMD:R_0603_1608Metric, F.Cu at (318.0, 574.0)
- added R812: 100k 0.1%, Resistor_SMD:R_0603_1608Metric, F.Cu at (350.0, 574.0)
- added R813: 10k 0.1%, Resistor_SMD:R_0603_1608Metric, F.Cu at (382.0, 574.0)
- added R814: 100, Resistor_SMD:R_0603_1608Metric, F.Cu at (414.0, 574.0)
- added R821: 100k 0.1%, Resistor_SMD:R_0603_1608Metric, F.Cu at (446.0, 574.0)
- added R822: 100k 0.1%, Resistor_SMD:R_0603_1608Metric, F.Cu at (478.0, 574.0)
- added R823: 10k 0.1%, Resistor_SMD:R_0603_1608Metric, F.Cu at (510.0, 574.0)
- added R824: 100, Resistor_SMD:R_0603_1608Metric, F.Cu at (542.0, 574.0)
- added R831: 100k 0.1%, Resistor_SMD:R_0603_1608Metric, F.Cu at (574.0, 574.0)
- added R832: 100k 0.1%, Resistor_SMD:R_0603_1608Metric, F.Cu at (30.0, 606.0)
- added R833: 10k 0.1%, Resistor_SMD:R_0603_1608Metric, F.Cu at (62.0, 606.0)
- added R834: 100, Resistor_SMD:R_0603_1608Metric, F.Cu at (94.0, 606.0)
- added R850: 8.2k, Resistor_SMD:R_0603_1608Metric, F.Cu at (126.0, 606.0)
- added R851: 10k, Resistor_SMD:R_0603_1608Metric, F.Cu at (158.0, 606.0)
- added R855: 8.2k, Resistor_SMD:R_0603_1608Metric, F.Cu at (190.0, 606.0)
- added R856: 10k, Resistor_SMD:R_0603_1608Metric, F.Cu at (222.0, 606.0)
- added R865: 1k, Resistor_SMD:R_0603_1608Metric, F.Cu at (254.0, 606.0)
- added R866: 10k, Resistor_SMD:R_0603_1608Metric, F.Cu at (286.0, 606.0)
- added R868: 1k, Resistor_SMD:R_0603_1608Metric, F.Cu at (318.0, 606.0)
- added R869: 10k, Resistor_SMD:R_0603_1608Metric, F.Cu at (350.0, 606.0)
- added R871: 1k, Resistor_SMD:R_0603_1608Metric, F.Cu at (382.0, 606.0)
- added R872: 10k, Resistor_SMD:R_0603_1608Metric, F.Cu at (414.0, 606.0)
- added R880: 10k 0.1%, Resistor_SMD:R_0603_1608Metric, F.Cu at (446.0, 606.0)
- added R883: 10k 0.1%, Resistor_SMD:R_0603_1608Metric, F.Cu at (478.0, 606.0)
- added R886: 10k 0.1%, Resistor_SMD:R_0603_1608Metric, F.Cu at (510.0, 606.0)
- added R887: 1k, Resistor_SMD:R_0603_1608Metric, F.Cu at (542.0, 606.0)
- added R889: 10k 0.1%, Resistor_SMD:R_0603_1608Metric, F.Cu at (574.0, 606.0)
- added R890: 1k, Resistor_SMD:R_0603_1608Metric, F.Cu at (30.0, 638.0)
- added R898: 10k 0.1%, Resistor_SMD:R_0603_1608Metric, F.Cu at (62.0, 638.0)
- added R899: 10k 0.1%, Resistor_SMD:R_0603_1608Metric, F.Cu at (94.0, 638.0)
- added SW501: RESET, Button_Switch_SMD:SW_SPST_TL3342, F.Cu at (126.0, 638.0)
- added SW502: USER, Button_Switch_SMD:SW_SPST_TL3342, F.Cu at (158.0, 638.0)
- added TH801: 10k / B25-50=3380K, Resistor_SMD:R_0603_1608Metric, F.Cu at (190.0, 638.0)
- added TH802: 10k / B25-50=3380K, Resistor_SMD:R_0603_1608Metric, F.Cu at (222.0, 638.0)
- added TP101: VBUS, TestPoint:TestPoint_Pad_D1.5mm, F.Cu at (254.0, 638.0)
- added TP102: GND, TestPoint:TestPoint_Pad_D1.5mm, F.Cu at (286.0, 638.0)
- added TP103: PHASE_A, TestPoint:TestPoint_Pad_D1.5mm, F.Cu at (318.0, 638.0)
- added TP104: PHASE_B, TestPoint:TestPoint_Pad_D1.5mm, F.Cu at (350.0, 638.0)
- added TP105: PHASE_C, TestPoint:TestPoint_Pad_D1.5mm, F.Cu at (382.0, 638.0)
- added TP210: I_PHASE_A, TestPoint:TestPoint_Pad_D1.5mm, F.Cu at (414.0, 638.0)
- added TP211: I_PHASE_B, TestPoint:TestPoint_Pad_D1.5mm, F.Cu at (446.0, 638.0)
- added TP212: I_PHASE_C, TestPoint:TestPoint_Pad_D1.5mm, F.Cu at (478.0, 638.0)
- added TP301: DUMP_CURRENT, TestPoint:TestPoint_Pad_D1.5mm, F.Cu at (510.0, 638.0)
- added TP401: 5V_BUS, TestPoint:TestPoint_Pad_D1.5mm, F.Cu at (542.0, 638.0)
- added TP402: 5V_SYS, TestPoint:TestPoint_Pad_D1.5mm, F.Cu at (574.0, 638.0)
- added TP403: 3V3, TestPoint:TestPoint_Pad_D1.5mm, F.Cu at (30.0, 670.0)
- added TP404: GND, TestPoint:TestPoint_Pad_D1.5mm, F.Cu at (62.0, 670.0)
- added TP501: VREF_3V0, TestPoint:TestPoint_Pad_D1.5mm, F.Cu at (94.0, 670.0)
- added TP502: VBIAS_1V5, TestPoint:TestPoint_Pad_D1.5mm, F.Cu at (126.0, 670.0)
- added TP503: 3V3_A, TestPoint:TestPoint_Pad_D1.5mm, F.Cu at (158.0, 670.0)
- added TP504: ADC_TRIG_SCOPE, TestPoint:TestPoint_Pad_D1.5mm, F.Cu at (190.0, 670.0)
- added TP505: DAC1_CH1_TP, TestPoint:TestPoint_Pad_D1.5mm, F.Cu at (222.0, 670.0)
- added TP506: DAC1_CH2_TP, TestPoint:TestPoint_Pad_D1.5mm, F.Cu at (254.0, 670.0)
- added U101: TLV1704IPWR, Package_SO:TSSOP-14_4.4x5mm_P0.65mm, F.Cu at (286.0, 670.0)
- added U102: TLV1704IPWR, Package_SO:TSSOP-14_4.4x5mm_P0.65mm, F.Cu at (318.0, 670.0)
- added U201: DRV8353SRTAT, bldc-esc:DRV8353_RTA0040B, F.Cu at (350.0, 670.0)
- added U202: INA241A2DR, Package_SO:SOIC-8_3.9x4.9mm_P1.27mm, F.Cu at (382.0, 670.0)
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
Commit message: devlog 03
Parts:
- removed D701, D702: BAT54H, Diode_SMD:D_SOD-123F
- added C312: 100p 50V, Capacitor_SMD:C_0603_1608Metric, F.Cu at (382.0, 734.0)
- added C313: 100n 50V, Capacitor_SMD:C_0603_1608Metric, F.Cu at (414.0, 734.0)
- added C314: 1u 16V, Capacitor_SMD:C_0603_1608Metric, F.Cu at (446.0, 734.0)
- added C706: 1u 16V, Capacitor_SMD:C_0603_1608Metric, F.Cu at (478.0, 734.0)
- added C847: 100n 50V, Capacitor_SMD:C_0603_1608Metric, F.Cu at (510.0, 734.0)
- added C848: 100n 50V, Capacitor_SMD:C_0603_1608Metric, F.Cu at (542.0, 734.0)
- added C852: 1n 50V, Capacitor_SMD:C_0603_1608Metric, F.Cu at (574.0, 734.0)
- added C857: 1n 50V, Capacitor_SMD:C_0603_1608Metric, F.Cu at (30.0, 766.0)
- added C888: 1n 50V, Capacitor_SMD:C_0603_1608Metric, F.Cu at (62.0, 766.0)
- added C891: 1n 50V, Capacitor_SMD:C_0603_1608Metric, F.Cu at (94.0, 766.0)
- added D704: PESD5V0S1BA, Diode_SMD:D_SOD-323, F.Cu at (126.0, 766.0)
- added D852: PESD5V0S1BA, Diode_SMD:D_SOD-323, F.Cu at (158.0, 766.0)
- added D857: PESD5V0S1BA, Diode_SMD:D_SOD-323, F.Cu at (190.0, 766.0)
- added D888: PESD5V0S1BA, Diode_SMD:D_SOD-323, F.Cu at (222.0, 766.0)
- added D891: PESD5V0S1BA, Diode_SMD:D_SOD-323, F.Cu at (254.0, 766.0)
- added R320: 10k 0.1%, Resistor_SMD:R_0603_1608Metric, F.Cu at (286.0, 766.0)
- added R321: 15k 0.1%, Resistor_SMD:R_0603_1608Metric, F.Cu at (318.0, 766.0)
- added R707: 100k, Resistor_SMD:R_0603_1608Metric, F.Cu at (350.0, 766.0)
- added R708: 100k, Resistor_SMD:R_0603_1608Metric, F.Cu at (382.0, 766.0)
- added R709: 1k, Resistor_SMD:R_0603_1608Metric, F.Cu at (414.0, 766.0)
- added R723: 10k, Resistor_SMD:R_0603_1608Metric, F.Cu at (446.0, 766.0)
- added R724: 100k, Resistor_SMD:R_0603_1608Metric, F.Cu at (478.0, 766.0)
- added R725: 100k, Resistor_SMD:R_0603_1608Metric, F.Cu at (510.0, 766.0)
- added R852: 100, Resistor_SMD:R_0603_1608Metric, F.Cu at (542.0, 766.0)
- added R857: 100, Resistor_SMD:R_0603_1608Metric, F.Cu at (574.0, 766.0)
- added R888: 100, Resistor_SMD:R_0603_1608Metric, F.Cu at (30.0, 798.0)
- added R891: 100, Resistor_SMD:R_0603_1608Metric, F.Cu at (62.0, 798.0)
- added TP220: GAH, TestPoint:TestPoint_Pad_D1.5mm, F.Cu at (94.0, 798.0)
- added TP221: GAL, TestPoint:TestPoint_Pad_D1.5mm, F.Cu at (126.0, 798.0)
- added TP222: SOURCE_A, TestPoint:TestPoint_Pad_D1.5mm, F.Cu at (158.0, 798.0)
- added TP240: GBH, TestPoint:TestPoint_Pad_D1.5mm, F.Cu at (190.0, 798.0)
- added TP241: GBL, TestPoint:TestPoint_Pad_D1.5mm, F.Cu at (222.0, 798.0)
- added TP242: SOURCE_B, TestPoint:TestPoint_Pad_D1.5mm, F.Cu at (254.0, 798.0)
- added TP260: GCH, TestPoint:TestPoint_Pad_D1.5mm, F.Cu at (286.0, 798.0)
- added TP261: GCL, TestPoint:TestPoint_Pad_D1.5mm, F.Cu at (318.0, 798.0)
- added TP262: SOURCE_C, TestPoint:TestPoint_Pad_D1.5mm, F.Cu at (350.0, 798.0)
- added U308: REF2025AIDDCR, Package_TO_SOT_SMD:SOT-23-5, F.Cu at (382.0, 798.0)
- added U803: TLV9062IDR, Package_SO:SOIC-8_3.9x4.9mm_P1.27mm, F.Cu at (414.0, 798.0)
- added U804: TLV9062IDR, Package_SO:SOIC-8_3.9x4.9mm_P1.27mm, F.Cu at (446.0, 798.0)
- C303: value 1n 50V -> 100n 50V
- C308: value 100p 50V -> 1n 50V
- C401, C402: footprint Capacitor_SMD:C_1206_3216Metric -> Capacitor_SMD:C_1210_3225Metric
- D301: value STPS5H100B -> STPS5H100AF; footprint Diode_SMD:D_SMC -> Diode_SMD:D_SOD-128
- D801, D811, D821, D831, D850, D855, D886, D889: value BAT54S -> BAV199
- J401: footprint Connector_USB:USB_C_Receptacle_GCT_USB4105-xx-A_16P_TopMnt_Horizontal -> bldc-esc:USB4105_PCBWay
- L401: value 68uH / Isat>=1.8A -> 68uH / Isat>=2.3A
- R316, R318: value 100k -> 150k
- R415: value 100k -> 10k
- R416: value 150k -> 15k
- R701, R703: value 10k -> 0
- U101, U102: value TLV1704IPWR -> TLV9024PWR
- U403: value TLV75533PDBVR -> TLV75533PDRVR; footprint Package_TO_SOT_SMD:SOT-23-5 -> Package_SON:WSON-6-1EP_2x2mm_P0.65mm_EP1x1.6mm
- U711, U712: value SN74LVC1G08DBVR -> SN74LVC1G11DBVR; footprint Package_TO_SOT_SMD:SOT-23-5 -> Package_TO_SOT_SMD:SOT-23-6
- Y501: footprint Crystal:Crystal_SMD_3225-4Pin_3.2x2.5mm -> Crystal:Crystal_SMD_Abracon_ABM3-2Pin_5.0x3.2mm
Connections:
- net /03_regen/BRK_CLEAR renamed /15_regen_safety/BRK_CLEAR
- net /03_regen/BRK_CLK renamed /15_regen_safety/BRK_CLK
- net /03_regen/BRK_CLK_RC renamed /15_regen_safety/BRK_CLK_RC
- net /03_regen/BRK_CT renamed /15_regen_safety/BRK_CT
- net /03_regen/BRK_OC_OK renamed /15_regen_safety/BRK_OC_OK
- net /03_regen/BRK_POR renamed /15_regen_safety/BRK_POR
- net /03_regen/DUMP_CURRENT renamed DUMP_CURRENT
- net /03_regen/nBRK_ARMED renamed /15_regen_safety/nBRK_ARMED
- net /03_regen/nDUMP_REQUEST renamed nDUMP_REQUEST
- net /08_analog_inputs/NTC_DUMP_IN renamed /14_temperature/NTC_DUMP_IN
- net /08_analog_inputs/NTC_MOTOR_IN renamed /14_temperature/NTC_MOTOR_IN
- net /09_safety/HW_ENABLE_OK renamed HW_ENABLE_OK
- net /09_safety/POR_CT renamed /16_supervisor/POR_CT
- net /09_safety/POWER_OK renamed /16_supervisor/POWER_OK
- net /09_safety/WD_CWD renamed /16_supervisor/WD_CWD
- net /09_safety/WD_OK renamed /16_supervisor/WD_OK
- net /09_safety/nHW_ENABLE_IN renamed /16_supervisor/nHW_ENABLE_IN
- C303 pad 1: /03_regen/DUMP_REF -> DUMP_REF
- C705 pad 1: nHW_ENABLE_SENSE -> nHW_ENABLE_FILT
- C850 pad 1: THROTTLE_ADC -> /08_analog_inputs/THROTTLE_ADC_DIV
- C855 pad 1: AUX_ANALOG_ADC -> /08_analog_inputs/AUX_ANALOG_ADC_DIV
- C886 pad 1: NTC_MOTOR -> /14_temperature/NTC_MOTOR_DIV
- C889 pad 1: NTC_DUMP -> /14_temperature/NTC_DUMP_DIV
- D850 pad 3: THROTTLE_ADC -> /08_analog_inputs/THROTTLE_ADC_DIV
- D855 pad 3: AUX_ANALOG_ADC -> /08_analog_inputs/AUX_ANALOG_ADC_DIV
- D886 pad 3: NTC_MOTOR -> /14_temperature/NTC_MOTOR_DIV
- D889 pad 3: NTC_DUMP -> /14_temperature/NTC_DUMP_DIV
- R304 pad 1: /03_regen/DUMP_REF -> DUMP_REF
- R314 pad 1: /03_regen/BRK_ARMED -> BRK_ARMED
- R621 pad 1: 3V3 -> 5V_HALL
- R624 pad 1: 3V3 -> 5V_HALL
- R627 pad 1: 3V3 -> 5V_HALL
- R633 pad 1: 3V3 -> 5V_ENCODER
- R636 pad 1: 3V3 -> 5V_ENCODER
- R639 pad 1: 3V3 -> 5V_ENCODER
- R701 pad 1: 3V3 -> NRST
- R703 pad 1: 3V3 -> NRST
- R721 pad 2: nHW_ENABLE_SENSE -> nHW_ENABLE_FILT
- R850 pad 2: THROTTLE_ADC -> /08_analog_inputs/THROTTLE_ADC_DIV
- R851 pad 1: THROTTLE_ADC -> /08_analog_inputs/THROTTLE_ADC_DIV
- R855 pad 2: AUX_ANALOG_ADC -> /08_analog_inputs/AUX_ANALOG_ADC_DIV
- R856 pad 1: AUX_ANALOG_ADC -> /08_analog_inputs/AUX_ANALOG_ADC_DIV
- R886 pad 2: NTC_MOTOR -> /14_temperature/NTC_MOTOR_DIV
- R887 pad 2: NTC_MOTOR -> /14_temperature/NTC_MOTOR_DIV
- R889 pad 2: NTC_DUMP -> /14_temperature/NTC_DUMP_DIV
- R890 pad 2: NTC_DUMP -> /14_temperature/NTC_DUMP_DIV
- U301 pad 5: /03_regen/DUMP_REF -> unconnected-(U301-REF-Pad5)
- U302 pad 6: /03_regen/BRK_ARMED -> BRK_ARMED
- U304 pad 3: /03_regen/DUMP_REF -> DUMP_REF
- U307 pad 5: /03_regen/BRK_ARMED -> BRK_ARMED
- U403 pad 1: 5V_SYS -> 3V3
- U403 pad 2: GND -> unconnected-(U403-NC-Pad2)
- U403 pad 3: 5V_SYS -> GND
- U403 pad 4: unconnected-(U403-NC-Pad4) -> 5V_SYS
- U403 pad 5: 3V3 -> unconnected-(U403-NC-Pad5)
- U501 pad 28: unconnected-(U501-PA6-Pad28) -> DUMP_I_ADC
- U501 pad 46: nFAULT_LATCH -> nFAULT_LATCH_SENSE
- U501 pad 68: BUS_OK -> BUS_OK_SENSE
- U501 pad 69: unconnected-(U501-PA8-Pad69) -> nOC_HW_SENSE
- U501 pad 91: DRV_nFAULT -> DRV_nFAULT_SENSE
- U501 pad 92: WD_RUN -> WD_RUN_SENSE
- U705 pad 5: nFAULT_LATCH -> /09_safety/nFAULT_LATCH
- U708 pad 6: nFAULT_LATCH -> /09_safety/nFAULT_LATCH
- U710 pad 2: nHW_ENABLE_SENSE -> nHW_ENABLE_FILT
- U711 pad 2: WD_RUN -> GND
- U711 pad 3: GND -> WD_RUN
- U712 pad 2: WD_RUN -> GND
- U712 pad 3: GND -> WD_RUN
- Y501 pad 2: GND -> /05_mcu/HSE_XOUT

Commit message: devlog 04
Parts:
- added C117: 10n 50V, Capacitor_SMD:C_0603_1608Metric, F.Cu at (574.0, 254.0)
- added R118: 40.2k 0.1%, Resistor_SMD:R_0603_1608Metric, F.Cu at (30.0, 286.0)
- added R119: 10k 0.1%, Resistor_SMD:R_0603_1608Metric, F.Cu at (478.0, 798.0)
- added R417: 51.1k 0.1%, Resistor_SMD:R_0603_1608Metric, F.Cu at (510.0, 798.0)
- added R418: 10k 0.1%, Resistor_SMD:R_0603_1608Metric, F.Cu at (542.0, 798.0)
- C410, C412, C506, C507: value 4.7u 10V -> 4.7u 25V
- C702: value 10n 50V -> 47n 50V
- F401: footprint Fuse:Fuse_1206_3216Metric -> bldc-esc:MF_PSMF0805
- J501: value SWD -> SWD / KEY 7; footprint Connector_PinHeader_1.27mm:PinHeader_2x05_P1.27mm_Vertical_SMD -> bldc-esc:FTSH_105_DV_007_K
- R111, R112: value 49.9k 0.1% -> 90.9k 0.1%
- R115: value 11k 0.1% -> 16.9k 0.1%
- R850, R855: value 8.2k -> 12.1k
- TP501: value VREF_3V0 -> VREF_2V5
- TP502: value VBIAS_1V5 -> VBIAS_1V25
- U202, U203, U204: value INA241A2DR -> INA241A2IDR
- U301: value TLV3011BDBVR -> TLV3011BIDBVR
- U403: value TLV75533PDRVR -> TLV75801PDRVR
- U502: value REF2030AIDDCR -> REF2025AIDDCR
- U701: value TPS3808G33DBVR -> TPS389033DSER; footprint Package_TO_SOT_SMD:SOT-23-6 -> Package_SON:WSON-6_1.5x1.5mm_P0.5mm
Connections:
- net VBIAS_1V5 renamed VBIAS_1V25
- net VREF_3V0 renamed VREF_2V5
- J101 pad 1: VBUS -> GND
- J101 pad 2: GND -> VBUS
- U102 pad 10: /11_current_protection/OC_LO -> /11_current_protection/BUS_UV_REF
- U403 pad 2: unconnected-(U403-NC-Pad2) -> /04_power_usb/VDD_FB
- U701 pad 1: /16_supervisor/POWER_OK -> 3V3_A
- U701 pad 4: /16_supervisor/POR_CT -> 3V3
- U701 pad 5: 3V3 -> /16_supervisor/POR_CT
- U701 pad 6: 3V3 -> /16_supervisor/POWER_OK

Commit message: devlog 05
Parts:
- moved R725 793.3 mm to (106.5, 83.0), turned to 90 degrees
- moved R418 787.7 mm to (106.0, 142.0), turned to 270 degrees
- moved R724 773.7 mm to (108.0, 86.5), turned to 90 degrees
- moved TP262 771.8 mm to (99.5, 68.0)
- moved R417 770.3 mm to (103.0, 144.0)
- moved R119 765.5 mm to (157.0, 103.0)
- moved U704 763.0 mm to (115.0, 92.5)
- moved TP260 761.8 mm to (99.0, 59.5)
- moved R857 758.3 mm to (134.5, 148.0), turned to 180 degrees
- moved TP261 757.8 mm to (106.0, 70.5)
- moved TP242 752.5 mm to (144.5, 53.5)
- moved U703 752.0 mm to (105.0, 90.0)
- moved U308 750.8 mm to (98.0, 103.0)
- moved TP240 748.4 mm to (113.5, 53.5)
- moved R723 745.5 mm to (109.0, 101.0)
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Other:
- board outline added: 116 x 112 mm
- board text added: "12-30 V"
- board text added: "AUX"
- board text added: "BLDC-ESC v1"
- board text added: "BRK DIR"
- board text added: "CAN"
- board text added: "ENC"
- board text added: "HALL"
- board text added: "RC"
- board text added: "TEMP M"
- board text added: "TEMP R"
- board text added: "THR"
- board text added: "UART"

Commit message: devlog 06
Parts:
- moved R304 7.67 mm to (99.4, 105.5)
- moved TP220 7.54 mm to (149.7, 50.6)
- moved TP103 6.05 mm to (153.4, 52.4)
- moved TP104 4.67 mm to (110.2, 53.2)
- moved C502 3.12 mm to (141.0, 106.6)
- moved TP242 1.75 mm to (144.4, 51.8)
- moved C504 1.24 mm to (121.8, 114.5)
- moved C515 1.03 mm to (144.5, 120.9)
- moved C511 0.76 mm to (130.8, 104.2)
- moved TP210 0.38 mm to (140.3, 103.7)
- turned C701 to 180 degrees
Routing:
- net VBUS: track 0.00 -> 331.8 mm, vias 0 -> 12
- net GND: track 0.00 -> 38.2 mm, vias 0 -> 31
- net nOC_HW: track 0.00 -> 30.7 mm
- net I_PHASE_A: track 0.00 -> 28.9 mm
- net 3V3: track 0.00 -> 25.1 mm, vias 0 -> 10
- net VREF_2V5: track 0.00 -> 24.2 mm, vias 0 -> 2
- net /11_current_protection/OC_LO: track 0.00 -> 22.4 mm, vias 0 -> 1
- net /11_current_protection/BUS_UV_REF: track 0.00 -> 21.0 mm
- net PHASE_A: track 0.00 -> 19.8 mm
- net /03_regen/DUMP_SW: track 0.00 -> 18.9 mm
- net /11_current_protection/OC_HI: track 0.00 -> 17.3 mm, vias 0 -> 1
- net 3V3_A: track 0.00 -> 16.9 mm, vias 0 -> 2
- net I_PHASE_B: track 0.00 -> 16.4 mm, vias 0 -> 4
- net I_DRV_B: track 0.00 -> 15.1 mm, vias 0 -> 1
- net I_DRV_A: track 0.00 -> 15.0 mm
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- added copper zone on In2.Cu, net 3V3
- added copper zone on B.Cu, net GND
- added copper zone on F.Cu, net GND
- added copper zone on In1.Cu, net GND
