File: bldc-esc.kicad_pcb (KiCad board)
At the start: 4 copper layers, 116 x 112 mm, 449 parts, among them J101 XT60PW-M, J102 MT60 / 12AWG pigtail, J103 CHASSIS, J301 DUMP RESISTOR, J401 USB4105-GF-A, J501 SWD / KEY 7, J601 HALL, J602 ENCODER, J701 CAN, J702 UART / 3V3, J703 HW ENABLE, J801 THROTTLE_ADC, J802 AUX_ANALOG_ADC, J803 RC PWM, J804 BRAKE / DIR, J805 NTC_MOTOR, J806 NTC_DUMP, Q201 ISC011N06LM5, Q202 ISC011N06LM5, Q203 ISC011N06LM5, Q204 ISC011N06LM5, Q205 ISC011N06LM5, Q206 ISC011N06LM5, Q301 ISC011N06LM5, Q302 2N7002, SW501 RESET, SW502 USER, U101 TLV9024PWR, U102 TLV9024PWR, U201 DRV8353SRTAT, U202 INA241A2IDR, U203 INA241A2IDR, U204 INA241A2IDR, U301 TLV3011BIDBVR, U302 UCC27511ADBVR, U303 INA180A1IDBVR, U304 TLV3201AIDBVR, U305 TPS3808G50DBVR, U306 SN74LVC1G17DBVR, U307 SN74LVC1G74DCTR, U308 REF2025AIDDCR, U401 LM5164DDAR, U402 TPS2116DRLR, U403 TLV75801PDRVR, U404 USBLC6-2SC6, U501 STM32G474VET6, U502 REF2025AIDDCR, U503 M24C64-RMN6TP, U601 TPS2553DBVR-1, U602 TPS2553DBVR-1, U603 SN74LVC3G17DCTR, U604 SN74LVC3G17DCTR, U701 TPS389033DSER, U702 TPS3431SDRBR, U703 SN74LVC1G11DBVR, U704 SN74LVC1G11DBVR, U705 SN74LVC1G74DCTR, U706 SN74LVC244APWR, U707 SN74LVC1G11DBVR, U708 SN74LVC1G11DBVR, U709 TCAN3403DRQ1, U710 SN74LVC1G14DBVR, U711 SN74LVC1G11DBVR, U712 SN74LVC1G11DBVR, U801 TLV9064IPWR, U802 SN74LVC3G17DCTR, U803 TLV9062IDR, U804 TLV9062IDR, Y501 8MHz / CL18p

Commit message: route buck converter and 5v feed
Parts:
- moved R406 10.6 mm to (69.0, 132.7), turned to 90 degrees
- moved R403 6.72 mm to (60.0, 140.2)
Routing:
- net 5V_BUS: track 15.2 -> 81.1 mm, vias 0 -> 7
- net VBUS: track 396.2 -> 448.6 mm, vias 146 -> 150
- net /04_power_usb/BUCK_RIPPLE: track 0.00 -> 20.7 mm, vias 0 -> 2
- net GND: track 132.1 -> 151.9 mm, vias 287 -> 300
- net /04_power_usb/BUS_5V_GOOD: track 0.00 -> 14.9 mm, vias 0 -> 2
- net /04_power_usb/BUCK_EN: track 0.00 -> 11.0 mm, vias 0 -> 2
- net /04_power_usb/BUCK_FB: track 0.00 -> 9.46 mm
- net /04_power_usb/BUCK_SW: track 0.00 -> 8.82 mm
- net /04_power_usb/BUCK_BST: track 0.00 -> 2.17 mm
- net /04_power_usb/BUCK_RON: track 0.00 -> 2.06 mm
- added copper zone on F.Cu, net /04_power_usb/BUCK_SW

Commit message: route usb power and logic supplies
Parts:
- moved R418 11.2 mm to (96.0, 137.0), turned to 0 degrees
- moved R417 6.40 mm to (99.0, 139.0), turned to 180 degrees
Routing:
- net USB_5V: track 0.00 -> 46.8 mm, vias 0 -> 2
- net 5V_SYS: track 0.00 -> 34.4 mm, vias 0 -> 2
- net 5V_BUS: track 81.1 -> 107.6 mm, vias 7 -> 9
- net /04_power_usb/MUX_PR1: track 0.00 -> 19.7 mm, vias 0 -> 2
- net /13_usb_status/USB_VBUS_RAW: track 0.00 -> 19.5 mm, vias 0 -> 3
- net /13_usb_status/CC2: track 0.00 -> 17.4 mm, vias 0 -> 2
- net GND: track 151.9 -> 167.2 mm, vias 300 -> 309
- net PWR_BUS_SELECTED: track 2.59 -> 15.0 mm, vias 1 -> 3
- net 3V3: track 25.1 -> 36.4 mm, vias 10 -> 15
- net /13_usb_status/CC1: track 0.00 -> 10.7 mm, vias 0 -> 2
- net /04_power_usb/VDD_FB: track 0.00 -> 9.76 mm, vias 0 -> 3
