File: schematic/04_power_usb.kicad_sch (KiCad schematic)
At the start: 26 parts, among them U401 LM5164DDAR, U402 TPS2116DRLR, U403 TLV75533PDRVR

Commit message: devlog 04
Parts:
- added R417: 51.1k 0.1%, Resistor_SMD:R_0603_1608Metric, symbol Device:R
- added R418: 10k 0.1%, Resistor_SMD:R_0603_1608Metric, symbol Device:R
- C401, C402: Manufacturer (none) -> TDK
- C403: MPN GCM188R71H222KA37D -> C0603C222J5GACTU; Manufacturer (none) -> KEMET
- C406, C407: Manufacturer (none) -> KEMET
- C408, C409, C411: MPN GRM188R71C105KA12D -> C0603C105K4RACTU; Manufacturer (none) -> KEMET
- C410, C412: value 4.7u 10V -> 4.7u 25V; MPN GRM21BR71A475KA73L -> C0805C475K3RACTU; Manufacturer (none) -> KEMET
- U403: value TLV75533PDRVR -> TLV75801PDRVR; symbol Regulator_Linear:TLV75533PDRV -> Regulator_Linear:TLV75801PDRV; MPN TLV75533PDRVR -> TLV75801PDRVR
Connections:
- net 3V3: now also R417.1
- net GND: now also R418.2
- net VDD_FB: now reaches U403.2 (FB)
- net VDD_FB: now also R417.2, R418.1
- no-connect marks 2 -> 1
Other:
- note added: "3V3 net: 3.3605 V nominal (51.1k / 10k). USB-only: bridge disarmed; sensor supplies off at boot."
- note added: "Bus / USB selection and logic supply"
- note removed: "Bus / USB selection and 3.3 V"
- note removed: "USB-only operation: bridge disarmed; sensor supplies disabled at boot."
- moved on the sheet: C410, C412, R410
