File: schematic/05_mcu.kicad_sch (KiCad schematic)
At the start: 0 parts

Commit message: devlog 02
Parts:
- added C501, C502, C503, C504, C505, C508, C509, C511, C512, C515, C516, C517: 100n 50V, Capacitor_SMD:C_0603_1608Metric, symbol Device:C
- added C506, C507: 4.7u 10V, Capacitor_SMD:C_0805_2012Metric, symbol Device:C
- added C510: 1u 16V, Capacitor_SMD:C_0603_1608Metric, symbol Device:C
- added C513, C514: 27p 50V, Capacitor_SMD:C_0603_1608Metric, symbol Device:C
- added D501: PMEG2010ER, Diode_SMD:Nexperia_CFP3_SOD-123W, symbol Device:D
- added FB501: 600R @ 100MHz, Inductor_SMD:L_0603_1608Metric, symbol Device:FerriteBead
- added J501: SWD, Connector_PinHeader_1.27mm:PinHeader_2x05_P1.27mm_Vertical_SMD, symbol Connector_Generic:Conn_02x05_Odd_Even
- added JP501: BOOT0, Connector_PinHeader_2.54mm:PinHeader_1x02_P2.54mm_Vertical, symbol Connector_Generic:Conn_01x02
- added R501: 1k, Resistor_SMD:R_0603_1608Metric, symbol Device:R
- added R502: 0, Resistor_SMD:R_0603_1608Metric, symbol Device:R
- added R503: 100k, Resistor_SMD:R_0603_1608Metric, symbol Device:R
- added R504, R505, R508: 10k, Resistor_SMD:R_0603_1608Metric, symbol Device:R
- added R506, R507: 4.7k, Resistor_SMD:R_0603_1608Metric, symbol Device:R
- added SW501: RESET, Button_Switch_SMD:SW_SPST_TL3342, symbol Switch:SW_Push
- added SW502: USER, Button_Switch_SMD:SW_SPST_TL3342, symbol Switch:SW_Push
- added TP501: VREF_3V0, TestPoint:TestPoint_Pad_D1.5mm, symbol Connector:TestPoint
- added TP502: VBIAS_1V5, TestPoint:TestPoint_Pad_D1.5mm, symbol Connector:TestPoint
- added TP503: 3V3_A, TestPoint:TestPoint_Pad_D1.5mm, symbol Connector:TestPoint
- added TP504: ADC_TRIG_SCOPE, TestPoint:TestPoint_Pad_D1.5mm, symbol Connector:TestPoint
- added TP505: DAC1_CH1_TP, TestPoint:TestPoint_Pad_D1.5mm, symbol Connector:TestPoint
- added TP506: DAC1_CH2_TP, TestPoint:TestPoint_Pad_D1.5mm, symbol Connector:TestPoint
- added U501: STM32G474VET6, Package_QFP:LQFP-100_14x14mm_P0.5mm, symbol MCU_ST_STM32G4:STM32G474VETx
- added U502: REF2030AIDDCR, Package_TO_SOT_SMD:SOT-23-5, symbol Reference_Voltage:REF2030
- added U503: M24C64-RMN6TP, Package_SO:SOIC-8_3.9x4.9mm_P1.27mm, symbol bldc-esc:M24C64_R
- added Y501: 8MHz / CL18p, Crystal:Crystal_SMD_3225-4Pin_3.2x2.5mm, symbol Device:Crystal_GND24
Connections:
- new net 3V3: C501.1, C502.1, C503.1, C504.1, C505.1, C506.1, C516.1, C517.1, FB501.1, J501.1 (Pin_1), JP501.2 (Pin_2), R504.1, R505.1, R506.1, R507.1, R508.1, U501.100 (VDD), U501.24 (VDD), U501.49 (VDD), U501.6 (VBAT), U501.64 (VDD), U501.75 (VDD), U503.8 (VCC)
- new net 3V3_A: C507.1, C508.1, C509.1, D501.1 (K), FB501.2, TP503.1, U501.37 (VDDA), U502.3 (EN), U502.4 (IN)
- new net ADC_TRIG_SCOPE: TP504.1, U501.45 (PE14)
- new net AUX_ANALOG_ADC: U501.18 (PC3)
- new net BOOT0: JP501.1 (Pin_1), R503.1, U501.95 (PB8)
- new net BRIDGE_ARM_REQ: U501.98 (PE1)
- new net BRK_FAULT_SENSE: U501.5 (PE6)
- new net BUS_OK: U501.68 (PC9)
- new net BUTTON_USER: R505.2, SW502.1, U501.7 (PC13)
- new net CAN_RX: U501.82 (PD0)
- new net CAN_STB: U501.71 (PA10)
- new net CAN_TX: U501.83 (PD1)
- new net DAC1_CH1_TP: TP505.1, U501.26 (PA4)
- new net DAC1_CH2_TP: TP506.1, U501.27 (PA5)
- new net DRV_SCK: U501.52 (PB13)
- new net DRV_SDI: U501.54 (PB15)
- new net DRV_SDO: U501.53 (PB14)
- new net DRV_WAKE_REQ: U501.81 (PC12)
- new net DRV_nCS: U501.51 (PB12)
- new net DRV_nFAULT: U501.91 (PB4)
- new net DUMP_ACTIVE_SENSE: U501.58 (PD11)
- new net DUMP_PWM: U501.97 (PE0)
- new net EEPROM_WP: R508.2, U501.94 (PB7), U503.7 (WC)
- new net ENCODER_5V_EN: U501.10 (PF9)
- new net ENCODER_nFAULT: U501.11 (PF10)
- new net ENC_A: U501.85 (PD3)
- new net ENC_B: U501.86 (PD4)
- new net ENC_Z: U501.89 (PD7)
- new net GND: C501.2, C502.2, C503.2, C504.2, C505.2, C506.2, C507.2, C508.2, C509.2, C510.2, C511.2, C512.2, C513.2, C514.2, C515.2, C516.2, C517.2, J501.3 (Pin_3), J501.5 (Pin_5), J501.9 (Pin_9), R501.2, R503.2, SW501.2, SW502.2, U501.23 (VSS), U501.35 (VSSA), U501.48 (VSS), U501.63 (VSS), U501.74 (VSS), U501.99 (VSS), U502.2 (GND), U503.1 (E0), U503.2 (E1), U503.3 (E2), U503.4 (VSS), Y501.2 (G), Y501.4 (G)
- new net HALL_1: U501.65 (PC6)
- new net HALL_2: U501.66 (PC7)
- new net HALL_3: U501.67 (PC8)
- new net HSE_IN: C513.1, U501.12 (PF0), Y501.1
- new net HSE_OUT: R502.1, U501.13 (PF1)
- new net HSE_XOUT: C514.1, R502.2, Y501.3
- new net I2C_SCL: R506.2, U501.78 (PA15), U503.6 (SCL)
- new net I2C_SDA: R507.2, U501.96 (PB9), U503.5 (SDA)
- new net I_DRV_A: U501.33 (PB1)
- new net I_DRV_B: U501.31 (PC5)
- new net I_DRV_C: U501.34 (PB2)
- new net I_PHASE_A: U501.16 (PC1), U501.21 (PA1)
- new net I_PHASE_B: U501.29 (PA7), U501.59 (PD12)
- new net I_PHASE_C: U501.32 (PB0), U501.50 (PB11)
- new net LED_COMM: U501.2 (PE3)
- new net LED_STATUS: U501.1 (PE2)
- new net NRST: C515.1, J501.10 (Pin_10), R504.2, SW501.1, U501.14 (PG10)
- new net NTC_BRIDGE: U501.55 (PD8)
- new net NTC_DUMP: U501.38 (PE7)
- new net NTC_MOTOR: U501.57 (PD10)
- new net NTC_PCB: U501.56 (PD9)
- new net PWM_AH: U501.40 (PE9)
- new net PWM_AL: U501.39 (PE8)
- new net PWM_BH: U501.42 (PE11)
- new net PWM_BL: U501.41 (PE10)
- new net PWM_CH: U501.44 (PE13)
- new net PWM_CL: U501.43 (PE12)
- new net PWR_BUS_SELECTED: U501.19 (PF2)
- new net RC_PWM_IN: U501.62 (PD15)
- new net SENSOR_5V_EN: U501.3 (PE4)
- new net SENSOR_nFAULT: U501.4 (PE5)
- new net SWCLK: J501.4 (Pin_4), U501.77 (PA14)
- new net SWDIO: J501.2 (Pin_2), U501.76 (PA13)
- new net SWO: J501.6 (Pin_6), U501.90 (PB3)
- new net THROTTLE_ADC: U501.17 (PC2)
- new net UART_RX: U501.80 (PC11)
- new net UART_TX: U501.79 (PC10)
- new net USB_DM: U501.72 (PA11)
- new net USB_DP: U501.73 (PA12)
- new net USB_VBUS_SENSE: U501.70 (PA9)
- new net VBIAS_1V5: C512.1, TP502.1, U502.1 (Vbias)
- new net VREF_3V0: C510.1, C511.1, D501.2 (A), R501.1, TP501.1, U501.36 (VREF+), U502.5 (Vref)
- new net V_3V3_ADC: U501.30 (PC4)
- new net V_BUS_ADC: U501.20 (PA0)
- new net V_PHASE_A: U501.22 (PA2)
- new net V_PHASE_B: U501.25 (PA3)
- new net V_PHASE_C: U501.15 (PC0)
- new net WD_HEARTBEAT: U501.84 (PD2)
- new net WD_RUN: U501.92 (PB5)
- new net nBRAKE_IN: U501.60 (PD13)
- new net nDIR_IN: U501.61 (PD14)
- new net nFAULT_LATCH: U501.46 (PE15)
- new net nHW_ENABLE_SENSE: U501.47 (PB10)
- no-connect marks 0 -> 9
Other:
- note added: "8 MHz crystal; load capacitors remain subject to startup validation."
- note added: "Injected ADC conversions use TIM1 TRGO. Configure break inputs, deadtime and safe GPIO states before requesting bridge arm."
- note added: "MCU bypass capacitors"
- note added: "MCU, reference and debug"
- note added: "Nonvolatile configuration"
- note added: "PB8 is BOOT0. PA15 carries I2C1 SCL."
- note added: "Programming / debug"
- note added: "STM32G474VET6 / TIM1 bridge control"
- note added: "VDDA and reference"
- note added: "VREF+ = 3.0 V; current midpoint = 1.5 V. Reference supply tracks VDDA during brownout."
- title: (none) -> MCU, reference and debug

Commit message: devlog 03
Parts:
- D501: Manufacturer (none) -> Nexperia
- Y501: footprint Crystal:Crystal_SMD_3225-4Pin_3.2x2.5mm -> Crystal:Crystal_SMD_Abracon_ABM3-2Pin_5.0x3.2mm; symbol Device:Crystal_GND24 -> Device:Crystal; MPN ABM8G-8.000MHZ-18-D2Y-T -> ABM3-8.000MHZ-D2Y-T
Connections:
- net GND: no longer Y501.2 (G), Y501.4 (G)
- net HSE_XOUT: now also Y501.2; no longer Y501.3
- net DUMP_I_ADC: now reaches U501.28 (PA6)
- net nOC_HW_SENSE: now reaches U501.69 (PA8)
- net BUS_OK renamed BUS_OK_SENSE
- net DRV_nFAULT renamed DRV_nFAULT_SENSE
- net WD_RUN renamed WD_RUN_SENSE
- net nFAULT_LATCH renamed nFAULT_LATCH_SENSE
- no-connect marks 9 -> 7
Other:
- moved on the sheet: C504, C505, C506, C507, C508, C509, C510, C511, C512, C516, C517, D501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

Commit message: devlog 04
Parts:
- C501, C502, C503, C504, C505, C508, C509, C511, C512, C515, C516, C517: MPN GRM188R71H104KA93D -> C0603C104K5RACTU; Manufacturer Murata -> KEMET
- C506, C507: value 4.7u 10V -> 4.7u 25V; MPN GRM21BR71A475KA73L -> C0805C475K3RACTU; Manufacturer (none) -> KEMET
- C510: MPN GRM188R71C105KA12D -> C0603C105K4RACTU; Manufacturer (none) -> KEMET
- C513, C514: Manufacturer (none) -> KEMET
- D501: MPN PMEG2010ER -> PMEG2010ER,115
- FB501: MPN BLM18AG601SN1D -> BLM18KG601SN1D
- J501: value SWD -> SWD / KEY 7; footprint Connector_PinHeader_1.27mm:PinHeader_2x05_P1.27mm_Vertical_SMD -> bldc-esc:FTSH_105_DV_007_K; symbol Connector_Generic:Conn_02x05_Odd_Even -> bldc-esc:SWD10_Keyed; MPN FTSH-105-01-L-DV-K -> FTSH-105-01-L-DV-007-K
- JP501: Manufacturer (none) -> Harwin
- TP501: value VREF_3V0 -> VREF_2V5
- TP502: value VBIAS_1V5 -> VBIAS_1V25
- U502: value REF2030AIDDCR -> REF2025AIDDCR; symbol Reference_Voltage:REF2030 -> Reference_Voltage:REF2025; MPN REF2030AIDDCR -> REF2025AIDDCR
Connections:
- net VBIAS_1V5 renamed VBIAS_1V25
- net VREF_3V0 renamed VREF_2V5
- no-connect marks 7 -> 6
Other:
- note added: "VREF+ = 2.5 V; current midpoint = 1.25 V. Reference supply tracks VDDA during brownout."
- note removed: "VREF+ = 3.0 V; current midpoint = 1.5 V. Reference supply tracks VDDA during brownout."
- moved on the sheet: C501, C502, C503, C504, C505, C506, C507, C508, C509, C510, C511, C512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
