File: schematic/06_sensors.kicad_sch (KiCad schematic)
At the start: 0 parts

Commit message: devlog 02
Parts:
- added C601, C603, C605, C606: 100n 50V, Capacitor_SMD:C_0603_1608Metric, symbol Device:C
- added C602, C604: 1u 16V, Capacitor_SMD:C_0603_1608Metric, symbol Device:C
- added C610, C611, C612, C613, C614, C615: 100p 50V, Capacitor_SMD:C_0603_1608Metric, symbol Device:C
- added D610, D611, D612, D613, D614, D615: PESD5V0S1BA, Diode_SMD:D_SOD-323, symbol Device:D_TVS
- added J601: HALL, Connector_JST:JST_GH_BM05B-GHS-TBT_1x05-1MP_P1.25mm_Vertical, symbol Connector_Generic:Conn_01x05
- added J602: ENCODER, Connector_JST:JST_GH_BM05B-GHS-TBT_1x05-1MP_P1.25mm_Vertical, symbol Connector_Generic:Conn_01x05
- added R601, R605: 200k, Resistor_SMD:R_0603_1608Metric, symbol Device:R
- added R602, R606: 100k, Resistor_SMD:R_0603_1608Metric, symbol Device:R
- added R603, R607, R621, R624, R627, R633, R636, R639: 10k, Resistor_SMD:R_0603_1608Metric, symbol Device:R
- added R620, R623, R626, R632, R635, R638: 1k, Resistor_SMD:R_0603_1608Metric, symbol Device:R
- added U601, U602: TPS2553DBVR-1, Package_TO_SOT_SMD:SOT-23-6, symbol bldc-esc:TPS2553_1
- added U603, U604: SN74LVC3G17DCTR, Package_SO:SSOP-8_2.95x2.8mm_P0.65mm, symbol bldc-esc:SN74LVC3G17
Connections:
- new net 3V3: C605.1, C606.1, R603.1, R607.1, R621.1, R624.1, R627.1, R633.1, R636.1, R639.1, U603.8 (VCC), U604.8 (VCC)
- new net 5V_ENCODER: C604.1, J602.1 (Pin_1), U602.6 (OUT)
- new net 5V_ENCODER_ILIM: R605.1, U602.5 (ILIM)
- new net 5V_HALL: C602.1, J601.1 (Pin_1), U601.6 (OUT)
- new net 5V_HALL_ILIM: R601.1, U601.5 (ILIM)
- new net 5V_SYS: C601.1, C603.1, U601.1 (IN), U602.1 (IN)
- new net ENCODER_5V_EN: R606.1, U602.3 (EN)
- new net ENCODER_nFAULT: R607.2, U602.4 (nFAULT)
- new net ENC_A: U604.7
- new net ENC_A_FILT: C613.1, R632.2, U604.1
- new net ENC_B: U604.5
- new net ENC_B_FILT: C614.1, R635.2, U604.3
- new net ENC_Z: U604.2
- new net ENC_Z_FILT: C615.1, R638.2, U604.6
- new net GND: C601.2, C602.2, C603.2, C604.2, C605.2, C606.2, C610.2, C611.2, C612.2, C613.2, C614.2, C615.2, D610.1 (A1), D610.2 (A2), D611.1 (A1), D611.2 (A2), D612.1 (A1), D612.2 (A2), D613.1 (A1), D613.2 (A2), D614.1 (A1), D614.2 (A2), D615.1 (A1), D615.2 (A2), J601.2 (Pin_2), J601.3 (Pin_3), J601.4 (Pin_4), J601.5 (Pin_5), J602.2 (Pin_2), J602.3 (Pin_3), J602.4 (Pin_4), J602.5 (Pin_5), R601.2, R602.2, R605.2, R606.2, R620.1, R621.2, R623.1, R624.2, R626.1, R627.2, R632.1, R633.2, R635.1, R636.2, R638.1, R639.2, U601.2 (GND), U602.2 (GND), U603.4 (GND), U604.4 (GND)
- new net HALL_1: U603.7
- new net HALL_1_FILT: C610.1, R620.2, U603.1
- new net HALL_2: U603.5
- new net HALL_2_FILT: C611.1, R623.2, U603.3
- new net HALL_3: U603.2
- new net HALL_3_FILT: C612.1, R626.2, U603.6
- new net SENSOR_5V_EN: R602.1, U601.3 (EN)
- new net SENSOR_nFAULT: R603.2, U601.4 (nFAULT)
Other:
- note added: "5 V supply: current limited, latch-off on fault. Inputs: 3.3/5 V single-ended, not 24 V."
- note added: "Connector labels define the controller pinout only. Verify the OEM motor Hall supply, ground and signal wires before connection."
- note added: "Encoder interface"
- note added: "Hall and encoder interfaces"
- note added: "Hall interface"
- title: (none) -> Hall and encoder interfaces

Commit message: devlog 03
Parts:
- D610, D611, D612, D613, D614, D615: Manufacturer (none) -> Nexperia
Connections:
- net 3V3: no longer R621.1, R624.1, R627.1, R633.1, R636.1, R639.1
- net 5V_ENCODER: now also R633.1, R636.1, R639.1
- net 5V_HALL: now also R621.1, R624.1, R627.1
Other:
- moved on the sheet: C602, C603, C604, C605, C606, C610, C611, C612, C613, C614, C615, D610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

Commit message: devlog 04
Parts:
- C601, C603, C605, C606: MPN GRM188R71H104KA93D -> C0603C104K5RACTU; Manufacturer Murata -> KEMET
- C602, C604: MPN GRM188R71C105KA12D -> C0603C105K4RACTU; Manufacturer (none) -> KEMET
- C610, C611, C612, C613, C614, C615: Manufacturer (none) -> KEMET
- D610, D611, D612, D613, D614, D615: MPN PESD5V0S1BA -> PESD5V0S1BA,115
