File: schematic/08_analog_inputs.kicad_sch (KiCad schematic)
At the start: 44 parts, among them J301 DUMP RESISTOR, Q301 ISC011N06LM5, Q302 2N7002, U301 TLV3011BDBVR, U302 UCC27511ADBVR, U303 INA180A1IDBVR, U304 TLV3201AIDBVR, U305 TPS3808G50DBVR, U306 SN74LVC1G17DBVR, U307 SN74LVC1G74DCTR

Commit message: devlog 02
Parts:
- removed C301, C303: 1n 50V, Capacitor_SMD:C_0603_1608Metric, symbol Device:C
- removed C302, C304, C306, C307, C309, C311: 100n 50V, Capacitor_SMD:C_0603_1608Metric, symbol Device:C
- removed C305: 1u 16V, Capacitor_SMD:C_0603_1608Metric, symbol Device:C
- removed C308: 100p 50V, Capacitor_SMD:C_0603_1608Metric, symbol Device:C
- removed C310: 10n 50V, Capacitor_SMD:C_0603_1608Metric, symbol Device:C
- removed D301: STPS5H100B, Diode_SMD:D_SMC, symbol Device:D
- removed D302, D303: BAT54H, Diode_SMD:D_SOD-123F, symbol Device:D
- removed J301: DUMP RESISTOR, TerminalBlock_Phoenix:TerminalBlock_Phoenix_MKDS-3-2-5.08_1x02_P5.08mm_Horizontal, symbol Connector_Generic:Conn_01x02
- removed Q301: ISC011N06LM5, Package_SON:Infineon_PG-TDSON-8_6.15x5.15mm, symbol bldc-esc:ISC011N06LM5
- removed Q302: 2N7002, Package_TO_SOT_SMD:SOT-23, symbol Transistor_FET:2N7002
- removed R301, R302: 100k 0.1%, Resistor_SMD:R_0603_1608Metric, symbol Device:R
- removed R303: 8.45k 0.1%, Resistor_SMD:R_0603_1608Metric, symbol Device:R
- removed R304: 10k 0.1%, Resistor_SMD:R_0603_1608Metric, symbol Device:R
- removed R305: 2.49M, Resistor_SMD:R_0603_1608Metric, symbol Device:R
- removed R306: 4.7k, Resistor_SMD:R_0603_1608Metric, symbol Device:R
- removed R307: 2.2, Resistor_SMD:R_0603_1608Metric, symbol Device:R
- removed R308: 1, Resistor_SMD:R_0603_1608Metric, symbol Device:R
- removed R309: 47k, Resistor_SMD:R_0603_1608Metric, symbol Device:R
- removed R310: 3m / 3W, Resistor_SMD:R_2512_6332Metric, symbol Device:R
- removed R311, R312, R313: 10k, Resistor_SMD:R_0603_1608Metric, symbol Device:R
- removed R314, R315, R316, R317, R318, R319: 100k, Resistor_SMD:R_0603_1608Metric, symbol Device:R
- removed TP301: DUMP_CURRENT, TestPoint:TestPoint_Pad_D1.5mm, symbol Connector:TestPoint
- removed U301: TLV3011BDBVR, Package_TO_SOT_SMD:SOT-23-6, symbol bldc-esc:TLV3011B
- removed U302: UCC27511ADBVR, Package_TO_SOT_SMD:SOT-23-6, symbol Driver_FET:UCC27511ADBV
- removed U303: INA180A1IDBVR, Package_TO_SOT_SMD:SOT-23-5, symbol Amplifier_Current:INA180A1
- removed U304: TLV3201AIDBVR, Package_TO_SOT_SMD:SOT-23-5, symbol bldc-esc:TLV3201
- removed U305: TPS3808G50DBVR, Package_TO_SOT_SMD:SOT-23-6, symbol bldc-esc:TPS3808Gxx
- removed U306: SN74LVC1G17DBVR, Package_TO_SOT_SMD:SOT-23-5, symbol 74xGxx:74LVC1G17
- removed U307: SN74LVC1G74DCTR, Package_SO:SSOP-8_2.95x2.8mm_P0.65mm, symbol bldc-esc:SN74LVC1G74
- added C845: 100n 50V, Capacitor_SMD:C_0603_1608Metric, symbol Device:C
- added C850, C855, C880, C883, C886, C889, C899: 10n 50V, Capacitor_SMD:C_0603_1608Metric, symbol Device:C
- added C865, C868, C871: 1n 50V, Capacitor_SMD:C_0603_1608Metric, symbol Device:C
- added D850, D855, D886, D889: BAT54S, Package_TO_SOT_SMD:SOT-23, symbol Diode:BAT54S
- added D865, D868, D871: PESD5V0S1BA, Diode_SMD:D_SOD-323, symbol Device:D_TVS
- added J801: THROTTLE_ADC, Connector_JST:JST_GH_BM03B-GHS-TBT_1x03-1MP_P1.25mm_Vertical, symbol Connector_Generic:Conn_01x03
- added J802: AUX_ANALOG_ADC, Connector_JST:JST_GH_BM03B-GHS-TBT_1x03-1MP_P1.25mm_Vertical, symbol Connector_Generic:Conn_01x03
- added J803: RC PWM, Connector_JST:JST_GH_BM03B-GHS-TBT_1x03-1MP_P1.25mm_Vertical, symbol Connector_Generic:Conn_01x03
- added J804: BRAKE / DIR, Connector_JST:JST_GH_BM03B-GHS-TBT_1x03-1MP_P1.25mm_Vertical, symbol Connector_Generic:Conn_01x03
- added J805: NTC_MOTOR, Connector_JST:JST_GH_BM02B-GHS-TBT_1x02-1MP_P1.25mm_Vertical, symbol Connector_Generic:Conn_01x02
- added J806: NTC_DUMP, Connector_JST:JST_GH_BM02B-GHS-TBT_1x02-1MP_P1.25mm_Vertical, symbol Connector_Generic:Conn_01x02
- added R850, R855: 8.2k, Resistor_SMD:R_0603_1608Metric, symbol Device:R
- added R851, R856, R866, R869, R872: 10k, Resistor_SMD:R_0603_1608Metric, symbol Device:R
- added R865, R868, R871, R887, R890: 1k, Resistor_SMD:R_0603_1608Metric, symbol Device:R
- added R880, R883, R886, R889, R898, R899: 10k 0.1%, Resistor_SMD:R_0603_1608Metric, symbol Device:R
- added TH801, TH802: 10k / B25-50=3380K, Resistor_SMD:R_0603_1608Metric, symbol Device:Thermistor_NTC
- added U802: SN74LVC3G17DCTR, Package_SO:SSOP-8_2.95x2.8mm_P0.65mm, symbol bldc-esc:SN74LVC3G17
Connections:
- net GND: now also C845.2, C850.2, C855.2, C865.2, C868.2, C871.2, C880.2, C883.2, C886.2, C889.2, C899.2, D850.1 (A), D855.1 (A), D865.1 (A1), D865.2 (A2), D868.1 (A1), D868.2 (A2), D871.1 (A1), D871.2 (A2), D886.1 (A), D889.1 (A), J801.2 (Pin_2), J802.2 (Pin_2), J803.1 (Pin_1), J803.3 (Pin_3), J804.1 (Pin_1), J804.2 (Pin_2), J804.3 (Pin_3), J805.2 (Pin_2), J806.2 (Pin_2), R851.2, R856.2, R865.1, R866.1, R866.2, R868.1, R869.2, R871.1, R872.2, R899.2, TH801.2, TH802.2, U802.4 (GND)
- new net 3V3: C845.1, R869.1, R872.1, R898.1, U802.8 (VCC)
- new net 3V3_A: D850.2 (K), D855.2 (K), D886.2 (K), D889.2 (K)
- new net 5V_HALL: J801.1 (Pin_1), J802.1 (Pin_1), J803.2 (Pin_2)
- new net AUX_ANALOG_ADC: C855.1, D855.3 (COM), R855.2, R856.1
- new net AUX_ANALOG_ADC_IN: J802.3 (Pin_3), R855.1
- new net NTC_BRIDGE: C880.1, R880.2, TH801.1
- new net NTC_DUMP: C889.1, D889.3 (COM), R889.2, R890.2
- new net NTC_DUMP_IN: J806.1 (Pin_1), R890.1
- new net NTC_MOTOR: C886.1, D886.3 (COM), R886.2, R887.2
- new net NTC_MOTOR_IN: J805.1 (Pin_1), R887.1
- new net NTC_PCB: C883.1, R883.2, TH802.1
- new net RC_PWM_IN: U802.7
- new net RC_PWM_RAW_FILT: C865.1, R865.2, U802.1
- new net THROTTLE_ADC: C850.1, D850.3 (COM), R850.2, R851.1
- new net THROTTLE_ADC_IN: J801.3 (Pin_3), R850.1
- new net VREF_3V0: R880.1, R883.1, R886.1, R889.1
- new net V_3V3_ADC: C899.1, R898.2, R899.1
- new net nBRAKE_IN: U802.5
- new net nBRAKE_RAW_FILT: C868.1, R868.2, U802.3
- new net nDIR_IN: U802.2
- new net nDIR_RAW_FILT: C871.1, R871.2, U802.6
- no-connect marks 1 -> 0
Other:
- note added: "Analog controls / 0-5 V input"
- note added: "Controls and temperature feedback"
- note added: "Digital controls / 3.3 or 5 V logic"
- note added: "TH801/TH802: 10k, B25/50=3380 K. External motor and dump-resistor NTCs use J805/J806. Validate all temperature conversions."
- note added: "Temperature feedback"
- note removed: "5 V-to-3.3 V monitor dividers"
- note removed: "Chopper overcurrent trip and power-cycle latch"
- note removed: "External dump resistor: 2-25 ohm; pulse/thermal rating required. Chopper trip: about 20.7 A, power-cycle reset."
- note removed: "Independent bus clamp / nominal 31.0 V on, 30.5 V off"
- note removed: "Regenerative brake chopper"
- note removed: "U302 return is Kelvin-connected to the top of R310. Do not force a bench supply to sink regenerative current."
- title: Regenerative brake chopper -> Controls and temperature feedback

Commit message: devlog 03
Parts:
- removed C880, C883, C886, C889, C899: 10n 50V, Capacitor_SMD:C_0603_1608Metric, symbol Device:C
- removed D886, D889: BAT54S, Package_TO_SOT_SMD:SOT-23, symbol Diode:BAT54S
- removed J805: NTC_MOTOR, Connector_JST:JST_GH_BM02B-GHS-TBT_1x02-1MP_P1.25mm_Vertical, symbol Connector_Generic:Conn_01x02
- removed J806: NTC_DUMP, Connector_JST:JST_GH_BM02B-GHS-TBT_1x02-1MP_P1.25mm_Vertical, symbol Connector_Generic:Conn_01x02
- removed R880, R883, R886, R889, R898, R899: 10k 0.1%, Resistor_SMD:R_0603_1608Metric, symbol Device:R
- removed R887, R890: 1k, Resistor_SMD:R_0603_1608Metric, symbol Device:R
- removed TH801, TH802: 10k / B25-50=3380K, Resistor_SMD:R_0603_1608Metric, symbol Device:Thermistor_NTC
- added C847: 100n 50V, Capacitor_SMD:C_0603_1608Metric, symbol Device:C
- added C852, C857: 1n 50V, Capacitor_SMD:C_0603_1608Metric, symbol Device:C
- added D852, D857: PESD5V0S1BA, Diode_SMD:D_SOD-323, symbol Device:D_TVS
- added R852, R857: 100, Resistor_SMD:R_0603_1608Metric, symbol Device:R
- added U803: TLV9062IDR, Package_SO:SOIC-8_3.9x4.9mm_P1.27mm, symbol bldc-esc:TLV9062
- D850, D855: value BAT54S -> BAV199; symbol Diode:BAT54S -> Device:D_Dual_Series_AKC; MPN BAT54S,215 -> BAV199,215
- D865, D868, D871: Manufacturer (none) -> Nexperia
Connections:
- net AUX_ANALOG_ADC_IN is gone; now on net GND: J802.3 (Pin_3), R855.1
- net THROTTLE_ADC_IN is gone; now on net GND: J801.3 (Pin_3), R850.1
- net 3V3_A: now also C847.1, U803.8 (V+)
- net AUX_ANALOG_ADC: now also C857.1, R857.2; no longer C855.1, D855.3 (COM), R855.2, R856.1
- net GND: now also C847.2, C852.2, C857.2, D852.1 (A1), D852.2 (A2), D857.1 (A1), D857.2 (A2), U803.4 (V-)
- net THROTTLE_ADC: now also C852.1, R852.2; no longer C850.1, D850.3 (COM), R850.2, R851.1
- new net AUX_ANALOG_ADC_BUF: R857.1, U803.6 (-), U803.7
- new net AUX_ANALOG_ADC_DIV: C855.1, D855.3 (common), R855.2, R856.1, U803.5 (+)
- new net THROTTLE_ADC_BUF: R852.1, U803.1, U803.2 (-)
- new net THROTTLE_ADC_DIV: C850.1, D850.3 (common), R850.2, R851.1, U803.3 (+)
Other:
- note added: "Analog and digital controls"
- note removed: "Controls and temperature feedback"
- note removed: "TH801/TH802: 10k, B25/50=3380 K. External motor and dump-resistor NTCs use J805/J806. Validate all temperature conversions."
- note removed: "Temperature feedback"
- title: Controls and temperature feedback -> Analog and digital controls
- moved on the sheet: C845, C850, C855, C865, C868, C871, D865, D868, D871, J802, J803, J804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

Commit message: devlog 04
Parts:
- C845, C847: MPN GRM188R71H104KA93D -> C0603C104K5RACTU; Manufacturer Murata -> KEMET
- C850, C852, C855, C857, C865, C868, C871: Manufacturer (none) -> KEMET
- D852, D857, D865, D868, D871: MPN PESD5V0S1BA -> PESD5V0S1BA,115
- R850, R855: value 8.2k -> 12.1k; MPN RC0603FR-078K2L -> RC0603FR-0712K1L
Other:
- moved on the sheet: C845, C847, C850, C852, C855, C857, C865, C868, C871, D850, D852, D855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
