File: schematic/09_safety.kicad_sch (KiCad schematic)
At the start: 45 parts, among them J703 HW ENABLE, U701 TPS3808G33DBVR, U702 TPS3431SDRBR, U703 SN74LVC1G11DBVR, U704 SN74LVC1G11DBVR, U705 SN74LVC1G74DCTR, U706 SN74LVC244APWR, U707 SN74LVC1G11DBVR, U708 SN74LVC1G11DBVR, U710 SN74LVC1G14DBVR, U711 SN74LVC1G08DBVR, U712 SN74LVC1G08DBVR

Commit message: devlog 03
Parts:
- removed C701, C703, C717, C718: 100n 50V, Capacitor_SMD:C_0603_1608Metric, symbol Device:C
- removed C702, C705: 10n 50V, Capacitor_SMD:C_0603_1608Metric, symbol Device:C
- removed D701, D702: BAT54H, Diode_SMD:D_SOD-123F, symbol Device:D
- removed J703: HW ENABLE, Connector_PinHeader_2.54mm:PinHeader_1x02_P2.54mm_Vertical, symbol Connector_Generic:Conn_01x02
- removed JP704: RUN 1-2 / SERVICE 2-3, Connector_PinHeader_2.54mm:PinHeader_1x03_P2.54mm_Vertical, symbol Connector_Generic:Conn_01x03
- removed R701, R702, R703, R720, R722: 10k, Resistor_SMD:R_0603_1608Metric, symbol Device:R
- removed R704: 100k, Resistor_SMD:R_0603_1608Metric, symbol Device:R
- removed R721: 1k, Resistor_SMD:R_0603_1608Metric, symbol Device:R
- removed U701: TPS3808G33DBVR, Package_TO_SOT_SMD:SOT-23-6, symbol bldc-esc:TPS3808Gxx
- removed U702: TPS3431SDRBR, Package_SON:VSON-8-1EP_3x3mm_P0.65mm_EP1.65x2.4mm, symbol bldc-esc:TPS3431
- removed U710: SN74LVC1G14DBVR, Package_TO_SOT_SMD:SOT-23-5, symbol 74xGxx:74LVC1G14
- added R707, R708, R724, R725: 100k, Resistor_SMD:R_0603_1608Metric, symbol Device:R
- added R709: 1k, Resistor_SMD:R_0603_1608Metric, symbol Device:R
- added R723: 10k, Resistor_SMD:R_0603_1608Metric, symbol Device:R
- U711, U712: value SN74LVC1G08DBVR -> SN74LVC1G11DBVR; footprint Package_TO_SOT_SMD:SOT-23-5 -> Package_TO_SOT_SMD:SOT-23-6; symbol 74xGxx:74LVC1G08 -> 74xGxx:74LVC1G11; MPN SN74LVC1G08DBVR -> SN74LVC1G11DBVR
Connections:
- net BUS_OK: now also R708.1
- net DRV_nFAULT: now also R725.1
- net GND: now also U711.2 (GND), U712.2 (GND); no longer U711.3 (GND), U712.3 (GND)
- net WD_RUN: now also U711.3, U712.3, R723.1; no longer U711.2, U712.2
- net nFAULT_LATCH: now also R709.1
- net nHW_ENABLE_SENSE: now also R724.2
- net nOC_HW: now also R707.1
- new net BRK_ARMED: U711.6, U712.6
- new net BUS_OK_SENSE: R708.2
- new net DRV_nFAULT_SENSE: R725.2
- new net WD_RUN_SENSE: R723.2
- new net nFAULT_LATCH_SENSE: R709.2
- new net nHW_ENABLE_FILT: R724.1
- new net nOC_HW_SENSE: R707.2
- no-connect marks 4 -> 2
Other:
- note added: "Hardware fault and enable nodes are isolated from MCU GPIO drive. Disable UCPD dead-battery control before reading PB4."
- note added: "MCU monitoring / series isolation"
- note removed: "Power-on reset and watchdog"
- note removed: "RUN 1-2 / SERVICE 2-3. SERVICE disables watchdog and forces both driver-enable and bridge-arm paths off."
- note removed: "Service and hardware enable"
- moved on the sheet: C711, C712, C713, C714, C715, C716, C719, C720, R705, R706, R710, R711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

Commit message: devlog 04
Parts:
- C711, C712, C713, C714, C715, C716, C719, C720: MPN GRM188R71H104KA93D -> C0603C104K5RACTU; Manufacturer Murata -> KEMET
