File: schematic/10_voltage_sensing.kicad_sch (KiCad schematic)
At the start: 26 parts, among them U401 LM5164DDAR, U402 TPS2116DRLR, U403 TLV75533PDBVR

Commit message: devlog 02
Parts:
- removed C401, C402: 2.2u 100V, Capacitor_SMD:C_1206_3216Metric, symbol Device:C
- removed C403, C406: 2.2n 50V, Capacitor_SMD:C_0603_1608Metric, symbol Device:C
- removed C404, C405: 22u 25V, Capacitor_SMD:C_1210_3225Metric, symbol Device:C
- removed C407: 82p 50V, Capacitor_SMD:C_0603_1608Metric, symbol Device:C
- removed C408, C409, C411: 1u 16V, Capacitor_SMD:C_0603_1608Metric, symbol Device:C
- removed C410, C412: 4.7u 10V, Capacitor_SMD:C_0805_2012Metric, symbol Device:C
- removed L401: 68uH / Isat>=1.8A, Inductor_SMD:L_Coilcraft_MSS1246T-XXX, symbol Device:L
- removed R401, R408: 300k, Resistor_SMD:R_0603_1608Metric, symbol Device:R
- removed R402, R409: 100k, Resistor_SMD:R_0603_1608Metric, symbol Device:R
- removed R403: 42.2k, Resistor_SMD:R_0603_1608Metric, symbol Device:R
- removed R404: 324k 0.1%, Resistor_SMD:R_0603_1608Metric, symbol Device:R
- removed R405: 100k 0.1%, Resistor_SMD:R_0603_1608Metric, symbol Device:R
- removed R406: 301k, Resistor_SMD:R_0603_1608Metric, symbol Device:R
- removed R407, R410: 10k, Resistor_SMD:R_0603_1608Metric, symbol Device:R
- removed U401: LM5164DDAR, Package_SO:HSOP-8-1EP_3.9x4.9mm_P1.27mm_EP2.41x3.1mm_ThermalVias, symbol Regulator_Switching:LM5164DDA
- removed U402: TPS2116DRLR, Package_TO_SOT_SMD:SOT-583-8, symbol Power_Management:TPS2116DRL
- removed U403: TLV75533PDBVR, Package_TO_SOT_SMD:SOT-23-5, symbol Regulator_Linear:TLV75533PDBV
- added C801, C811, C821, C831: 220p 50V, Capacitor_SMD:C_0603_1608Metric, symbol Device:C
- added C802, C812, C822, C832: 1n 50V, Capacitor_SMD:C_0603_1608Metric, symbol Device:C
- added C840: 100n 50V, Capacitor_SMD:C_0603_1608Metric, symbol Device:C
- added D801, D811, D821, D831: BAT54S, Package_TO_SOT_SMD:SOT-23, symbol Diode:BAT54S
- added R801, R802, R811, R812, R821, R822, R831, R832: 100k 0.1%, Resistor_SMD:R_0603_1608Metric, symbol Device:R
- added R803, R813, R823, R833: 10k 0.1%, Resistor_SMD:R_0603_1608Metric, symbol Device:R
- added R804, R814, R824, R834: 100, Resistor_SMD:R_0603_1608Metric, symbol Device:R
- added U801: TLV9064IPWR, Package_SO:TSSOP-14_4.4x5mm_P0.65mm, symbol bldc-esc:TLV9064
Connections:
- net GND: now also C801.2, C802.2, C811.2, C812.2, C821.2, C822.2, C831.2, C832.2, C840.2, D801.1 (A), D811.1 (A), D821.1 (A), D831.1 (A), R803.2, R813.2, R823.2, R833.2, U801.11 (V-)
- net VBUS: now also R801.1
- new net 3V3_A: C840.1, D801.2 (K), D811.2 (K), D821.2 (K), D831.2 (K), U801.4 (V+)
- new net PHASE_A: R811.1
- new net PHASE_B: R821.1
- new net PHASE_C: R831.1
- new net V_BUS_ADC: C802.1, R804.2
- new net V_BUS_ADC_BUF: R804.1, U801.1, U801.2 (-)
- new net V_BUS_ADC_DIV: C801.1, D801.3 (COM), R802.2, R803.1, U801.3 (+)
- new net V_BUS_ADC_MID: R801.2, R802.1
- new net V_PHASE_A: C812.1, R814.2
- new net V_PHASE_A_BUF: R814.1, U801.6 (-), U801.7
- new net V_PHASE_A_DIV: C811.1, D811.3 (COM), R812.2, R813.1, U801.5 (+)
- new net V_PHASE_A_MID: R811.2, R812.1
- new net V_PHASE_B: C822.1, R824.2
- new net V_PHASE_B_BUF: R824.1, U801.8, U801.9 (-)
- new net V_PHASE_B_DIV: C821.1, D821.3 (COM), R822.2, R823.1, U801.10 (+)
- new net V_PHASE_B_MID: R821.2, R822.1
- new net V_PHASE_C: C832.1, R834.2
- new net V_PHASE_C_BUF: R834.1, U801.13 (-), U801.14
- new net V_PHASE_C_DIV: C831.1, D831.3 (COM), R832.2, R833.1, U801.12 (+)
- new net V_PHASE_C_MID: R831.2, R832.1
- no-connect marks 1 -> 0
Other:
- note added: "21:1 dividers; 3.0 V ADC full scale = 63 V at the input. Buffers isolate the dividers from ADC sampling transients. Normal operation remains limited to a 12-30 V bus."
- note added: "Bus and phase voltage sensing"
- note added: "Bus voltage"
- note added: "Phase A voltage"
- note added: "Phase B voltage"
- note added: "Phase C voltage"
- note removed: "68 uH / about 300 kHz. R406, C406, C407 provide type-3 ripple injection. Verify startup and load transients."
- note removed: "Bus / USB selection and 3.3 V"
- note removed: "Bus supply / LM5164, nominal 5 V"
- note removed: "Power supplies and USB"
- note removed: "USB-only operation: bridge disarmed; sensor supplies disabled at boot."
- title: Power supplies and USB -> Bus and phase voltage sensing

Commit message: devlog 03
Parts:
- D801, D811, D821, D831: value BAT54S -> BAV199; symbol Diode:BAT54S -> Device:D_Dual_Series_AKC; MPN BAT54S,215 -> BAV199,215
Other:
- moved on the sheet: C801, C802, C811, C812, C821, C822, C831, C832, R801, R802, R803, R804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

Commit message: devlog 04
Parts:
- C801, C802, C811, C812, C821, C822, C831, C832: Manufacturer (none) -> KEMET
- C840: MPN GRM188R71H104KA93D -> C0603C104K5RACTU; Manufacturer Murata -> KEMET
Other:
- note added: "21:1 dividers; 2.5 V ADC full scale = 52.5 V at the input. Buffers isolate the dividers from ADC sampling transients. Normal operation remains limited to a 12-30 V bus."
- note removed: "21:1 dividers; 3.0 V ADC full scale = 63 V at the input. Buffers isolate the dividers from ADC sampling transients. Normal operation remains limited to a 12-30 V bus."
- moved on the sheet: C840
Changed lines of the file:
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@@
     )
   )
-  (text "21:1 dividers; 3.0 V ADC full scale = 63 V at the input.\nBuffers isolate the dividers from ADC sampling transients.\nNormal operation remains limited to a 12-30 V bus."
-    (at 82.55 189.23 0)
+  (text "21:1 dividers; 2.5 V ADC full scale = 52.5 V at the input.\nBuffers isolate the dividers from ADC sampling transients.\nNormal operation remains limited to a 12-30 V bus."
+    (at 90.17 189.23 0)
     (effects
       (font
@@
       (hide yes)
     )
-    (property "Manufacturer" ""
+    (property "Manufacturer" "KEMET"
       (at 97.79 63.5 0)
       (effects
@@
       (hide yes)
     )
-    (property "Manufacturer" ""
+    (property "Manufacturer" "KEMET"
       (at 168.91 66.04 0)
       (effects
@@
       (hide yes)
     )
-    (property "Manufacturer" ""
+    (property "Manufacturer" "KEMET"
       (at 273.05 63.5 0)
       (effects
@@
       (hide yes)
     )
-    (property "Manufacturer" ""
+    (property "Manufacturer" "KEMET"
       (at 344.17 66.04 0)
       (effects
@@
       (hide yes)
     )
-    (property "Manufacturer" ""
+    (property "Manufacturer" "KEMET"
       (at 102.87 139.7 0)
       (effects
@@
       (hide yes)
     )
-    (property "Manufacturer" ""
+    (property "Manufacturer" "KEMET"
       (at 173.99 142.24 0)
       (effects
@@
       (hide yes)
     )
-    (property "Manufacturer" ""
+    (property "Manufacturer" "KEMET"
       (at 276.86 139.7 0)
       (effects
@@
       (hide yes)
     )
-    (property "Manufacturer" ""
+    (property "Manufacturer" "KEMET"
       (at 347.98 142.24 0)
       (effects
@@
     (dnp no)
     (property "Reference" "U801"
-      (at 19.05 189.23 0)
+      (at 22.86 191.77 0)
       (effects
         (font
           (size 1.15 1.15)
         )
+        (justify left)
       )
     )
     (property "Value" "TLV9064IPWR"
-      (at 19.05 191.77 0)
+      (at 22.86 194.31 0)
       (effects
         (font
           (size 1.15 1.15)
         )
+        (justify left)
       )
     )
@@
           (size 1.15 1.15)
         )
+        (justify left)
       )
       (hide yes)
@@
           (size 1.15 1.15)
         )
+        (justify left)
       )
       (hide yes)
@@
           (size 1.15 1.15)
         )
+        (justify left)
       )
       (hide yes)
@@
           (size 1.15 1.15)
         )
+        (justify left)
       )
       (hide yes)
@@
   (symbol
     (lib_id "Device:C")
-    (at 31.75 199.39 0)
+    (at 39.37 199.39 0)
     (unit 1)
     (exclude_from_sim no)
@@
     (dnp no)
     (property "Reference" "C840"
-      (at 35.56 196.85 0)
+      (at 43.18 196.85 0)
       (effects
         (font
@@
     )
     (property "Value" "100n 50V"
-      (at 35.56 199.39 0)
+      (at 43.18 199.39 0)
       (effects
         (font
@@
     )
     (property "Footprint" "Capacitor_SMD:C_0603_1608Metric"
-      (at 31.75 199.39 0)
+      (at 39.37 199.39 0)
       (effects
         (font
@@
     )
     (property "Datasheet" ""
-      (at 31.75 199.39 0)
+      (at 39.37 199.39 0)
       (effects
         (font
@@
       (hide yes)
     )
-    (property "MPN" "GRM188R71H104KA93D"
-      (at 31.75 199.39 0)
+    (property "MPN" "C0603C104K5RACTU"
+      (at 39.37 199.39 0)
       (effects
         (font
@@
       (hide yes)
     )
-    (property "Manufacturer" "Murata"
-      (at 31.75 199.39 0)
+    (property "Manufacturer" "KEMET"
+      (at 39.37 199.39 0)
       (effects
         (font
@@
   (symbol
     (lib_id "power:VCC")
-    (at 31.75 190.5 0)
+    (at 39.37 190.5 0)
     (unit 1)
     (exclude_from_sim no)
@@
     (dnp no)
     (property "Reference" "#PWR100001"
-      (at 31.75 190.5 0)
+      (at 39.37 190.5 0)
       (effects
         (font
@@
     )
     (property "Value" "3V3_A"
-      (at 31.75 186.69 0)
+      (at 39.37 186.69 0)
       (effects
         (font
@@
   (symbol
     (lib_id "power:GND")
-    (at 31.75 208.28 0)
+    (at 39.37 208.28 0)
     (unit 1)
     (exclude_from_sim no)
@@
     (dnp no)
     (property "Reference" "#PWR100002"
-      (at 31.75 208.28 0)
+      (at 39.37 208.28 0)
       (effects
         (font
@@
     )
     (property "Value" "GND"
-      (at 31.75 212.09 0)
+      (at 39.37 212.09 0)
       (effects
         (font
@@
   (wire
     (pts
-      (xy 31.75 190.5)
-      (xy 31.75 195.58)
+      (xy 39.37 190.5)
+      (xy 39.37 195.58)
     )
     (stroke
@@
   (wire
     (pts
-      (xy 31.75 203.2)
-      (xy 31.75 208.28)
+      (xy 39.37 203.2)
+      (xy 39.37 208.28)
     )
     (stroke
