File: schematic/11_current_protection.kicad_sch (KiCad schematic)
At the start: 15 parts, among them U101 TLV1704IPWR, U102 TLV1704IPWR

Commit message: devlog 03
Parts:
- U101, U102: value TLV1704IPWR -> TLV9024PWR; symbol bldc-esc:TLV1704 -> bldc-esc:TLV9024; MPN TLV1704IPWR -> TLV9024PWR
Other:
- moved on the sheet: C112, C113, C114, R114, R115, R116, R117, U101A, U101B, U101C, U101D, U102A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

Commit message: devlog 04
Parts:
- added C117: 10n 50V, Capacitor_SMD:C_0603_1608Metric, symbol Device:C
- added R118: 40.2k 0.1%, Resistor_SMD:R_0603_1608Metric, symbol Device:R
- added R119: 10k 0.1%, Resistor_SMD:R_0603_1608Metric, symbol Device:R
- C110, C111, C112: Manufacturer (none) -> KEMET
- C113, C114: MPN GRM188R71H104KA93D -> C0603C104K5RACTU; Manufacturer Murata -> KEMET
- R111, R112: value 49.9k 0.1% -> 90.9k 0.1%; MPN RT0603BRD0749K9L -> RT0603BRD0790K9L
- R115: value 11k 0.1% -> 16.9k 0.1%; MPN RT0603BRD0711KL -> RT0603BRD0716K9L
Connections:
- net GND: now also C117.2, R119.2
- net OC_LO: no longer U102.10 (-)
- net VREF_3V0 renamed VREF_2V5
- net VREF_2V5: now also R118.1
- new net BUS_UV_REF: C117.1, R118.2, R119.1, U102.10 (-)
Other:
- moved on the sheet: C110, C111, C112, C113, C114, R110, R111, R112, R113, R114, R115, R117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
