File: schematic/12_gate_driver.kicad_sch (KiCad schematic)
At the start: 13 parts, among them U201 DRV8353SRTAT

Commit message: devlog 03
Parts:
- C201: MPN UPW1J220MED -> EEUFC1J220; Manufacturer Nichicon -> Panasonic
Changed lines of the file:
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@@
       (hide yes)
     )
-    (property "Datasheet" ""
+    (property "Datasheet" "https://industrial.panasonic.com/sa/products/pt/aluminum-cap-lead/models/EEUFC1J220"
       (at 50.8 63.5 0)
       (effects
@@
       (hide yes)
     )
-    (property "MPN" "UPW1J220MED"
+    (property "MPN" "EEUFC1J220"
       (at 50.8 63.5 0)
       (effects
@@
       (hide yes)
     )
-    (property "Manufacturer" "Nichicon"
+    (property "Manufacturer" "Panasonic"
       (at 50.8 63.5 0)
       (effects
@@
   )
   (symbol
+    (lib_id "power:VCC")
+    (at 31.75 101.6 0)
+    (unit 1)
+    (exclude_from_sim no)
+    (in_bom no)
+    (on_board yes)
+    (dnp no)
+    (property "Reference" "#PWR120001"
+      (at 31.75 101.6 0)
+      (effects
+        (font
+          (size 1.0 1.0)
+        )
+        (hide yes)
+      )
+    )
+    (property "Value" "VBUS"
+      (at 31.75 97.79 0)
+      (effects
+        (font
+          (size 1.0 1.0)
+        )
+      )
+    )
+    (instances
+      (project "bldc-esc"
+        (path "/10000000-0000-4000-8000-000000000000/10000000-0000-4000-8000-000000000012"
+          (reference "#PWR120001")
+          (unit 1)
+        )
+      )
+    )
+  )
+  (symbol
+    (lib_id "power:VCC")
+    (at 39.37 104.14 0)
+    (unit 1)
+    (exclude_from_sim no)
+    (in_bom no)
+    (on_board yes)
+    (dnp no)
+    (property "Reference" "#PWR120002"
+      (at 39.37 104.14 0)
+      (effects
+        (font
+          (size 1.0 1.0)
+        )
+        (hide yes)
+      )
+    )
+    (property "Value" "3V3_A"
+      (at 39.37 100.33 0)
+      (effects
+        (font
+          (size 1.0 1.0)
+        )
+      )
+    )
+    (instances
+      (project "bldc-esc"
+        (path "/10000000-0000-4000-8000-000000000000/10000000-0000-4000-8000-000000000012"
+          (reference "#PWR120002")
+          (unit 1)
+        )
+      )
+    )
+  )
+  (symbol
     (lib_id "power:GND")
     (at 50.8 72.39 0)
@@
     (on_board yes)
     (dnp no)
-    (property "Reference" "#PWR120001"
+    (property "Reference" "#PWR120003"
       (at 50.8 72.39 0)
       (effects
@@
       (project "bldc-esc"
         (path "/10000000-0000-4000-8000-000000000000/10000000-0000-4000-8000-000000000012"
-          (reference "#PWR120001")
+          (reference "#PWR120003")
           (unit 1)
         )
@@
     (on_board yes)
     (dnp no)
-    (property "Reference" "#PWR120002"
+    (property "Reference" "#PWR120004"
       (at 71.12 72.39 0)
       (effects
@@
       (project "bldc-esc"
         (path "/10000000-0000-4000-8000-000000000000/10000000-0000-4000-8000-000000000012"
-          (reference "#PWR120002")
+          (reference "#PWR120004")
           (unit 1)
         )
@@
     (on_board yes)
     (dnp no)
-    (property "Reference" "#PWR120003"
+    (property "Reference" "#PWR120005"
       (at 139.7 115.57 0)
       (effects
@@
       (project "bldc-esc"
         (path "/10000000-0000-4000-8000-000000000000/10000000-0000-4000-8000-000000000012"
-          (reference "#PWR120003")
+          (reference "#PWR120005")
           (unit 1)
         )
@@
     (on_board yes)
     (dnp no)
-    (property "Reference" "#PWR120004"
+    (property "Reference" "#PWR120006"
       (at 139.7 148.59 0)
       (effects
@@
       (project "bldc-esc"
         (path "/10000000-0000-4000-8000-000000000000/10000000-0000-4000-8000-000000000012"
-          (reference "#PWR120004")
+          (reference "#PWR120006")
           (unit 1)
         )
@@
     (on_board yes)
     (dnp no)
-    (property "Reference" "#PWR120005"
+    (property "Reference" "#PWR120007"
       (at 30.48 130.81 0)
       (effects
@@
       (project "bldc-esc"
         (path "/10000000-0000-4000-8000-000000000000/10000000-0000-4000-8000-000000000012"
-          (reference "#PWR120005")
+          (reference "#PWR120007")
           (unit 1)
         )
@@
     (on_board yes)
     (dnp no)
-    (property "Reference" "#PWR120006"
+    (property "Reference" "#PWR120008"
       (at 43.18 147.32 0)
       (effects
@@
       (project "bldc-esc"
         (path "/10000000-0000-4000-8000-000000000000/10000000-0000-4000-8000-000000000012"
-          (reference "#PWR120006")
-          (unit 1)
-        )
-      )
-    )
-  )
-  (symbol
-    (lib_id "power:VCC")
-    (at 46.99 101.6 0)
-    (unit 1)
-    (exclude_from_sim no)
-    (in_bom no)
-    (on_board yes)
-    (dnp no)
-    (property "Reference" "#PWR120007"
-      (at 46.99 101.6 0)
-      (effects
-        (font
-          (size 1.0 1.0)
-        )
-        (hide yes)
-      )
-    )
-    (property "Value" "VBUS"
-      (at 46.99 97.79 0)
-      (effects
-        (font
-          (size 1.0 1.0)
-        )
-      )
-    )
-    (instances
-      (project "bldc-esc"
-        (path "/10000000-0000-4000-8000-000000000000/10000000-0000-4000-8000-000000000012"
-          (reference "#PWR120007")
-          (unit 1)
-        )
-      )
-    )
-  )
-  (symbol
-    (lib_id "power:VCC")
-    (at 46.99 104.14 0)
-    (unit 1)
-    (exclude_from_sim no)
-    (in_bom no)
-    (on_board yes)
-    (dnp no)
-    (property "Reference" "#PWR120008"
-      (at 46.99 104.14 0)
-      (effects
-        (font
-          (size 1.0 1.0)
-        )
-        (hide yes)
-      )
-    )
-    (property "Value" "3V3_A"
-      (at 46.99 100.33 0)
-      (effects
-        (font
-          (size 1.0 1.0)
-        )
-      )
-    )
-    (instances
-      (project "bldc-esc"
-        (path "/10000000-0000-4000-8000-000000000000/10000000-0000-4000-8000-000000000012"
           (reference "#PWR120008")
           (unit 1)
@@
   (wire
     (pts
-      (xy 46.99 104.14)
+      (xy 39.37 104.14)
       (xy 52.07 104.14)
     )
@@
   (wire
     (pts
+      (xy 24.13 99.06)
+      (xy 52.07 99.06)
+    )
+    (stroke
+      (width 0)
+      (type default)
+    )
+  )
+  (wire
+    (pts
       (xy 30.48 76.2)
       (xy 30.48 81.28)
@@
   (wire
     (pts
-      (xy 46.99 99.06)
-      (xy 52.07 99.06)
-    )
-    (stroke
-      (width 0)
-      (type default)
-    )
-  )
-  (wire
-    (pts
       (xy 50.8 48.26)
       (xy 50.8 59.69)
@@
   (wire
     (pts
-      (xy 46.99 101.6)
+      (xy 31.75 101.6)
       (xy 52.07 101.6)
     )
@@
     (diameter 0)
     (color 0 0 0 0)
+  )
+  (label "DRV_VM"
+    (at 24.13 99.06 0)
+    (effects
+      (font
+        (size 0.95 0.95)
+      )
+      (justify right bottom)
+    )
   )
   (label "DRV_VM"
@@
     )
   )
-  (label "DRV_VM"
-    (at 46.99 99.06 0)
-    (effects
-      (font
-        (size 0.95 0.95)
-      )
-      (justify right bottom)
-    )
-  )

Commit message: devlog 04
Parts:
- C202: MPN GRM188R72A104KA35D -> C0603C104K1RACTU; Manufacturer (none) -> KEMET
- C203: MPN GRM21BR72A473KA01L -> C0805C473K1RACTU; Manufacturer (none) -> KEMET
- C204: Manufacturer (none) -> TDK
- C205: MPN GRM21BR71E105KA99L -> C0805C105K3RACTU; Manufacturer (none) -> KEMET
- C206: MPN GRM188R71C105KA12D -> C0603C105K4RACTU; Manufacturer (none) -> KEMET
- C207: MPN GRM188R71H104KA93D -> C0603C104K5RACTU; Manufacturer Murata -> KEMET
Changed lines of the file:
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@@
       (hide yes)
     )
-    (property "MPN" "GRM188R72A104KA35D"
+    (property "MPN" "C0603C104K1RACTU"
       (at 71.12 63.5 0)
       (effects
@@
       (hide yes)
     )
-    (property "Manufacturer" ""
+    (property "Manufacturer" "KEMET"
       (at 71.12 63.5 0)
       (effects
@@
       (hide yes)
     )
-    (property "MPN" "GRM21BR72A473KA01L"
+    (property "MPN" "C0805C473K1RACTU"
       (at 137.16 55.88 0)
       (effects
@@
       (hide yes)
     )
-    (property "Manufacturer" ""
+    (property "Manufacturer" "KEMET"
       (at 137.16 55.88 0)
       (effects
@@
       (hide yes)
     )
-    (property "Manufacturer" ""
+    (property "Manufacturer" "TDK"
       (at 154.94 78.74 0)
       (effects
@@
       (hide yes)
     )
-    (property "MPN" "GRM21BR71E105KA99L"
+    (property "MPN" "C0805C105K3RACTU"
       (at 139.7 106.68 0)
       (effects
@@
       (hide yes)
     )
-    (property "Manufacturer" ""
+    (property "Manufacturer" "KEMET"
       (at 139.7 106.68 0)
       (effects
@@
       (hide yes)
     )
-    (property "MPN" "GRM188R71C105KA12D"
+    (property "MPN" "C0603C105K4RACTU"
       (at 139.7 139.7 0)
       (effects
@@
       (hide yes)
     )
-    (property "Manufacturer" ""
+    (property "Manufacturer" "KEMET"
       (at 139.7 139.7 0)
       (effects
@@
       (hide yes)
     )
-    (property "MPN" "GRM188R71H104KA93D"
+    (property "MPN" "C0603C104K5RACTU"
       (at 30.48 121.92 0)
       (effects
@@
       (hide yes)
     )
-    (property "Manufacturer" "Murata"
+    (property "Manufacturer" "KEMET"
       (at 30.48 121.92 0)
       (effects
