File: schematic/13_usb_status.kicad_sch (KiCad schematic)
At the start: 20 parts, among them J401 USB4105-GF-A, U404 USBLC6-2SC6

Commit message: devlog 04
Parts:
- C413: MPN GRM188R71H104KA93D -> C0603C104K5RACTU; Manufacturer Murata -> KEMET
- F401: footprint Fuse:Fuse_1206_3216Metric -> bldc-esc:MF_PSMF0805
Other:
- moved on the sheet: D511, D512, D513, R511, R512, R513, TP401, TP402, TP403, TP404
