File: schematic/14_temperature.kicad_sch (KiCad schematic)
At the start: 26 parts, among them U401 LM5164DDAR, U402 TPS2116DRLR, U403 TLV75533PDRVR

Commit message: devlog 03
Parts:
- removed C401, C402: 2.2u 100V, Capacitor_SMD:C_1210_3225Metric, symbol Device:C
- removed C403, C406: 2.2n 50V, Capacitor_SMD:C_0603_1608Metric, symbol Device:C
- removed C404, C405: 22u 25V, Capacitor_SMD:C_1210_3225Metric, symbol Device:C
- removed C407: 82p 50V, Capacitor_SMD:C_0603_1608Metric, symbol Device:C
- removed C408, C409, C411: 1u 16V, Capacitor_SMD:C_0603_1608Metric, symbol Device:C
- removed C410, C412: 4.7u 10V, Capacitor_SMD:C_0805_2012Metric, symbol Device:C
- removed L401: 68uH / Isat>=2.3A, Inductor_SMD:L_Coilcraft_MSS1246T-XXX, symbol Device:L
- removed R401, R408: 300k, Resistor_SMD:R_0603_1608Metric, symbol Device:R
- removed R402, R409: 100k, Resistor_SMD:R_0603_1608Metric, symbol Device:R
- removed R403: 42.2k, Resistor_SMD:R_0603_1608Metric, symbol Device:R
- removed R404: 324k 0.1%, Resistor_SMD:R_0603_1608Metric, symbol Device:R
- removed R405: 100k 0.1%, Resistor_SMD:R_0603_1608Metric, symbol Device:R
- removed R406: 301k, Resistor_SMD:R_0603_1608Metric, symbol Device:R
- removed R407, R410: 10k, Resistor_SMD:R_0603_1608Metric, symbol Device:R
- removed U401: LM5164DDAR, Package_SO:HSOP-8-1EP_3.9x4.9mm_P1.27mm_EP2.41x3.1mm_ThermalVias, symbol Regulator_Switching:LM5164DDA
- removed U402: TPS2116DRLR, Package_TO_SOT_SMD:SOT-583-8, symbol Power_Management:TPS2116DRL
- removed U403: TLV75533PDRVR, Package_SON:WSON-6-1EP_2x2mm_P0.65mm_EP1x1.6mm, symbol Regulator_Linear:TLV75533PDRV
- added C848: 100n 50V, Capacitor_SMD:C_0603_1608Metric, symbol Device:C
- added C880, C883, C886, C889, C899: 10n 50V, Capacitor_SMD:C_0603_1608Metric, symbol Device:C
- added C888, C891: 1n 50V, Capacitor_SMD:C_0603_1608Metric, symbol Device:C
- added D886, D889: BAV199, Package_TO_SOT_SMD:SOT-23, symbol Device:D_Dual_Series_AKC
- added D888, D891: PESD5V0S1BA, Diode_SMD:D_SOD-323, symbol Device:D_TVS
- added J805: NTC_MOTOR, Connector_JST:JST_GH_BM02B-GHS-TBT_1x02-1MP_P1.25mm_Vertical, symbol Connector_Generic:Conn_01x02
- added J806: NTC_DUMP, Connector_JST:JST_GH_BM02B-GHS-TBT_1x02-1MP_P1.25mm_Vertical, symbol Connector_Generic:Conn_01x02
- added R880, R883, R886, R889, R898, R899: 10k 0.1%, Resistor_SMD:R_0603_1608Metric, symbol Device:R
- added R887, R890: 1k, Resistor_SMD:R_0603_1608Metric, symbol Device:R
- added R888, R891: 100, Resistor_SMD:R_0603_1608Metric, symbol Device:R
- added TH801, TH802: 10k / B25-50=3380K, Resistor_SMD:R_0603_1608Metric, symbol Device:Thermistor_NTC
- added U804: TLV9062IDR, Package_SO:SOIC-8_3.9x4.9mm_P1.27mm, symbol bldc-esc:TLV9062
Connections:
- net 3V3: now also R898.1
- net GND: now also C848.2, C880.2, C883.2, C886.2, C888.2, C889.2, C891.2, C899.2, D886.1 (A), D888.1 (A1), D888.2 (A2), D889.1 (A), D891.1 (A1), D891.2 (A2), J805.1 (Pin_1), J805.2 (Pin_2), J806.1 (Pin_1), J806.2 (Pin_2), R887.1, R890.1, R899.2, TH801.2, TH802.2, U804.4 (V-)
- new net 3V3_A: C848.1, D886.2 (K), D889.2 (K), U804.8 (V+)
- new net NTC_BRIDGE: C880.1, R880.2, TH801.1
- new net NTC_DUMP: C891.1, R891.2
- new net NTC_DUMP_BUF: R891.1, U804.6 (-), U804.7
- new net NTC_DUMP_DIV: C889.1, D889.3 (common), R889.2, R890.2, U804.5 (+)
- new net NTC_MOTOR: C888.1, R888.2
- new net NTC_MOTOR_BUF: R888.1, U804.1, U804.2 (-)
- new net NTC_MOTOR_DIV: C886.1, D886.3 (common), R886.2, R887.2, U804.3 (+)
- new net NTC_PCB: C883.1, R883.2, TH802.1
- new net VREF_3V0: R880.1, R883.1, R886.1, R889.1
- new net V_3V3_ADC: C899.1, R898.2, R899.1
- no-connect marks 2 -> 0
Other:
- note added: "TH801/TH802: 10k, B25/50=3380 K. External NTC conversion must subtract the 1k series resistor. External channels are buffered; configure their actual R/T curves before thermal-limit testing."
- note added: "Temperature and logic-rail feedback"
- note added: "Temperature feedback"
- note removed: "68 uH / about 300 kHz. R406, C406, C407 provide type-3 ripple injection. Verify startup and load transients."
- note removed: "Bus / USB selection and 3.3 V"
- note removed: "Bus supply / LM5164, nominal 5 V"
- note removed: "Power supplies"
- note removed: "USB-only operation: bridge disarmed; sensor supplies disabled at boot."
- title: Power supplies -> Temperature and logic-rail feedback

Commit message: devlog 04
Parts:
- C848: MPN GRM188R71H104KA93D -> C0603C104K5RACTU; Manufacturer Murata -> KEMET
- C880, C883, C886, C888, C889, C891, C899: Manufacturer (none) -> KEMET
- D888, D891: MPN PESD5V0S1BA -> PESD5V0S1BA,115
Connections:
- net VREF_3V0 renamed VREF_2V5
Other:
- moved on the sheet: C848, C886, C888, C889, C891, D886, D888, D889, D891, J805, J806, R886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
