File: schematic/15_regen_safety.kicad_sch (KiCad schematic)
At the start: 22 parts, among them U304 TLV3201AIDBVR, U305 TPS3808G50DBVR, U306 SN74LVC1G17DBVR, U307 SN74LVC1G74DCTR

Commit message: devlog 04
Parts:
- C307, C309, C311: MPN GRM188R71H104KA93D -> C0603C104K5RACTU; Manufacturer Murata -> KEMET
- C308, C310, C312: Manufacturer (none) -> KEMET
- D302, D303: MPN BAT54H -> BAT54H,115
Other:
- moved on the sheet: C312, R315, R316, R317, R318, R320, R321
