File: schematic/16_supervisor.kicad_sch (KiCad schematic)
At the start: 20 parts, among them J401 USB4105-GF-A, U404 USBLC6-2SC6

Commit message: devlog 03
Parts:
- removed C413: 100n 50V, Capacitor_SMD:C_0603_1608Metric, symbol Device:C
- removed D511: STATUS, LED_SMD:LED_0603_1608Metric, symbol Device:LED
- removed D512: COMM, LED_SMD:LED_0603_1608Metric, symbol Device:LED
- removed D513: POWER, LED_SMD:LED_0603_1608Metric, symbol Device:LED
- removed F401: 0.5A / 6V, Fuse:Fuse_1206_3216Metric, symbol Device:Polyfuse
- removed J401: USB4105-GF-A, bldc-esc:USB4105_PCBWay, symbol bldc-esc:USB_C_16P
- removed R411, R412: 5.1k, Resistor_SMD:R_0603_1608Metric, symbol Device:R
- removed R413, R414: 22, Resistor_SMD:R_0603_1608Metric, symbol Device:R
- removed R415: 10k, Resistor_SMD:R_0603_1608Metric, symbol Device:R
- removed R416: 15k, Resistor_SMD:R_0603_1608Metric, symbol Device:R
- removed R511, R512, R513: 1k, Resistor_SMD:R_0603_1608Metric, symbol Device:R
- removed TP401: 5V_BUS, TestPoint:TestPoint_Pad_D1.5mm, symbol Connector:TestPoint
- removed TP402: 5V_SYS, TestPoint:TestPoint_Pad_D1.5mm, symbol Connector:TestPoint
- removed TP403: 3V3, TestPoint:TestPoint_Pad_D1.5mm, symbol Connector:TestPoint
- removed TP404: GND, TestPoint:TestPoint_Pad_D1.5mm, symbol Connector:TestPoint
- removed U404: USBLC6-2SC6, Package_TO_SOT_SMD:SOT-23-6, symbol Power_Protection:USBLC6-2SC6
- added C701, C703, C717, C718: 100n 50V, Capacitor_SMD:C_0603_1608Metric, symbol Device:C
- added C702, C705: 10n 50V, Capacitor_SMD:C_0603_1608Metric, symbol Device:C
- added D704: PESD5V0S1BA, Diode_SMD:D_SOD-323, symbol Device:D_TVS
- added J703: HW ENABLE, Connector_PinHeader_2.54mm:PinHeader_1x02_P2.54mm_Vertical, symbol Connector_Generic:Conn_01x02
- added JP704: RUN 1-2 / SERVICE 2-3, Connector_PinHeader_2.54mm:PinHeader_1x03_P2.54mm_Vertical, symbol Connector_Generic:Conn_01x03
- added R701, R703: 0, Resistor_SMD:R_0603_1608Metric, symbol Device:R
- added R702, R720, R722: 10k, Resistor_SMD:R_0603_1608Metric, symbol Device:R
- added R704: 100k, Resistor_SMD:R_0603_1608Metric, symbol Device:R
- added R721: 1k, Resistor_SMD:R_0603_1608Metric, symbol Device:R
- added U701: TPS3808G33DBVR, Package_TO_SOT_SMD:SOT-23-6, symbol bldc-esc:TPS3808Gxx
- added U702: TPS3431SDRBR, Package_SON:VSON-8-1EP_3x3mm_P0.65mm_EP1.65x2.4mm, symbol bldc-esc:TPS3431
- added U710: SN74LVC1G14DBVR, Package_TO_SOT_SMD:SOT-23-5, symbol 74xGxx:74LVC1G14
Connections:
- net 3V3: now also C701.1, C703.1, C717.1, C718.1, JP704.1 (Pin_1), R702.1, R720.1, R722.1, U701.3 (nMR), U701.5 (SENSE), U701.6 (VDD), U702.1 (VDD), U702.3 (EN), U710.5 (VCC)
- net GND: now also C701.2, C702.2, C703.2, C705.2, C717.2, C718.2, D704.1 (A1), D704.2 (A2), J703.1 (Pin_1), J703.2 (Pin_2), JP704.3 (Pin_3), R704.2, R720.2, R721.1, U701.2 (GND), U702.4 (GND), U702.9 (EP), U710.3 (GND)
- new net HW_ENABLE_OK: U710.4
- new net NRST: R701.1, R703.1
- new net POR_CT: C702.1, U701.4 (CT)
- new net POWER_OK: R701.2, U701.1 (nRESET)
- new net WD_CWD: R702.2, U702.2 (CWD)
- new net WD_HEARTBEAT: R704.1, U702.6 (WDI)
- new net WD_OK: R703.2, U702.7 (nWDO)
- new net WD_RUN: JP704.2 (Pin_2), R722.2, U702.5 (SET1)
- new net nHW_ENABLE_FILT: C705.1, R721.2, U710.2
Other:
- note added: "Open-drain reset outputs share NRST through zero-ohm links. R504 on the MCU sheet provides the pull-up."
- note added: "Power-on reset and watchdog"
- note added: "RUN 1-2 / SERVICE 2-3. SERVICE or a chopper fault forces both driver-enable and bridge-arm paths off."
- note added: "Reset, watchdog and hardware enable"
- note added: "Service and hardware enable"
- note removed: "Status / probe points"
- note removed: "USB and status indicators"
- note removed: "USB shield bonds to CHASSIS. D+/D- protection belongs close to the connector; 22 ohm resistors belong near the MCU."
- note removed: "USB-C device port"
- title: USB and status indicators -> Reset, watchdog and hardware enable

Commit message: devlog 04
Parts:
- C701, C703, C717, C718: MPN GRM188R71H104KA93D -> C0603C104K5RACTU; Manufacturer Murata -> KEMET
- C702: value 10n 50V -> 47n 50V; MPN C0603C103K5RACTU -> C0603C473K5RACTU; Manufacturer (none) -> KEMET
- C705: Manufacturer (none) -> KEMET
- D704: MPN PESD5V0S1BA -> PESD5V0S1BA,115
- J703, JP704: Manufacturer (none) -> Harwin
- U701: value TPS3808G33DBVR -> TPS389033DSER; footprint Package_TO_SOT_SMD:SOT-23-6 -> Package_SON:WSON-6_1.5x1.5mm_P0.5mm; symbol bldc-esc:TPS3808Gxx -> bldc-esc:TPS3890; MPN TPS3808G33DBVR -> TPS389033DSER
Connections:
- net 3V3: now also U701.4 (VDD); no longer U701.5 (SENSE), U701.6 (VDD)
- net POR_CT: now also U701.5 (CT); no longer U701.4 (CT)
- net POWER_OK: now also U701.6 (nRESET); no longer U701.1 (nRESET)
- new net 3V3_A: U701.1 (SENSE)
