File: schematic/02_bridge.kicad_sch (KiCad schematic)
At the start: 0 parts

Commit message: devlog 02
Parts:
- added C210, C211, C230, C231, C250, C251: 1u 100V, Capacitor_SMD:C_1206_3216Metric, symbol Device:C
- added C212, C232, C252: 100n 50V, Capacitor_SMD:C_0603_1608Metric, symbol Device:C
- added C213, C214, C233, C234, C253, C254: 1n 50V, Capacitor_SMD:C_0603_1608Metric, symbol Device:C
- added C215, C235, C255: 1n 100V, Capacitor_SMD:C_0805_2012Metric, symbol Device:C
- added Q201, Q202, Q203, Q204, Q205, Q206: ISC011N06LM5, Package_SON:Infineon_PG-TDSON-8_6.15x5.15mm, symbol bldc-esc:ISC011N06LM5
- added R210, R212, R230, R232, R250, R252: 3.3, Resistor_SMD:R_0603_1608Metric, symbol Device:R
- added R211, R213, R231, R233, R251, R253: 47k, Resistor_SMD:R_0603_1608Metric, symbol Device:R
- added R214, R234, R254: 1m 1% 8W, bldc-esc:CSS4J_4026, symbol Device:R_Shunt
- added R215, R235, R255: 100, Resistor_SMD:R_0603_1608Metric, symbol Device:R
- added R216, R236, R256: 1k, Resistor_SMD:R_0603_1608Metric, symbol Device:R
- added R217, R237, R257: 10, Resistor_SMD:R_0805_2012Metric, symbol Device:R
- added TP210: I_PHASE_A, TestPoint:TestPoint_Pad_D1.5mm, symbol Connector:TestPoint
- added TP211: I_PHASE_B, TestPoint:TestPoint_Pad_D1.5mm, symbol Connector:TestPoint
- added TP212: I_PHASE_C, TestPoint:TestPoint_Pad_D1.5mm, symbol Connector:TestPoint
- added U202, U203, U204: INA241A2DR, Package_SO:SOIC-8_3.9x4.9mm_P1.27mm, symbol Amplifier_Current:INA241A2xDGK
Connections:
- new net 3V3_A: C212.1, C232.1, C252.1, U202.6 (V+), U203.6 (V+), U204.6 (V+)
- new net GAH: Q201.4 (G), R210.2, R211.1
- new net GAL: Q202.4 (G), R212.2, R213.1
- new net GBH: Q203.4 (G), R230.2, R231.1
- new net GBL: Q204.4 (G), R232.2, R233.1
- new net GCH: Q205.4 (G), R250.2, R251.1
- new net GCL: Q206.4 (G), R252.2, R253.1
- new net GHA_DRV: R210.1
- new net GHB_DRV: R230.1
- new net GHC_DRV: R250.1
- new net GLA_DRV: R212.1
- new net GLB_DRV: R232.1
- new net GLC_DRV: R252.1
- new net GND: C210.2, C211.2, C212.2, C213.2, C214.2, C215.2, C230.2, C231.2, C232.2, C233.2, C234.2, C235.2, C250.2, C251.2, C252.2, C253.2, C254.2, C255.2, R214.4, R234.4, R254.4, U202.2 (GND), U202.4 (GND), U203.2 (GND), U203.4 (GND), U204.2 (GND), U204.4 (GND)
- new net I_A_RAW: R215.1, U202.5
- new net I_B_RAW: R235.1, U203.5
- new net I_C_RAW: R255.1, U204.5
- new net I_DRV_A: C214.1, R216.2
- new net I_DRV_B: C234.1, R236.2
- new net I_DRV_C: C254.1, R256.2
- new net I_PHASE_A: C213.1, R215.2, TP210.1
- new net I_PHASE_B: C233.1, R235.2, TP211.1
- new net I_PHASE_C: C253.1, R255.2, TP212.1
- new net KS_A_N: R214.3, U202.1 (-)
- new net KS_A_P: R214.2, U202.8 (+)
- new net KS_B_N: R234.3, U203.1 (-)
- new net KS_B_P: R234.2, U203.8 (+)
- new net KS_C_N: R254.3, U204.1 (-)
- new net KS_C_P: R254.2, U204.8 (+)
- new net PHASE_A: Q201.1 (S), Q201.2 (S), Q201.3 (S), Q202.5 (D), R211.2, R217.1
- new net PHASE_B: Q203.1 (S), Q203.2 (S), Q203.3 (S), Q204.5 (D), R231.2, R237.1
- new net PHASE_C: Q205.1 (S), Q205.2 (S), Q205.3 (S), Q206.5 (D), R251.2, R257.1
- new net SNUB_A: C215.1, R217.2
- new net SNUB_B: C235.1, R237.2
- new net SNUB_C: C255.1, R257.2
- new net SOURCE_A: Q202.1 (S), Q202.2 (S), Q202.3 (S), R213.2, R214.1
- new net SOURCE_B: Q204.1 (S), Q204.2 (S), Q204.3 (S), R233.2, R234.1
- new net SOURCE_C: Q206.1 (S), Q206.2 (S), Q206.3 (S), R253.2, R254.1
- new net SO_A_DRV: R216.1
- new net SO_B_DRV: R236.1
- new net SO_C_DRV: R256.1
- new net VBIAS_1V5: U202.3 (REF2), U202.7 (REF1), U203.3 (REF2), U203.7 (REF1), U204.3 (REF2), U204.7 (REF1)
- new net VBUS: C210.1, C211.1, C230.1, C231.1, C250.1, C251.1, Q201.5 (D), Q203.5 (D), Q205.5 (D)
Other:
- note added: "Main CSA: 1.5 V zero, 20 mV/A DRV CSA: diagnostic channel"
- note added: "Phase A"
- note added: "Phase B"
- note added: "Phase C"
- note added: "Three-phase bridge and current sensing"
- title: (none) -> Three-phase bridge and current sensing

Commit message: devlog 03
Parts:
- added TP220: GAH, TestPoint:TestPoint_Pad_D1.5mm, symbol Connector:TestPoint
- added TP221: GAL, TestPoint:TestPoint_Pad_D1.5mm, symbol Connector:TestPoint
- added TP222: SOURCE_A, TestPoint:TestPoint_Pad_D1.5mm, symbol Connector:TestPoint
- added TP240: GBH, TestPoint:TestPoint_Pad_D1.5mm, symbol Connector:TestPoint
- added TP241: GBL, TestPoint:TestPoint_Pad_D1.5mm, symbol Connector:TestPoint
- added TP242: SOURCE_B, TestPoint:TestPoint_Pad_D1.5mm, symbol Connector:TestPoint
- added TP260: GCH, TestPoint:TestPoint_Pad_D1.5mm, symbol Connector:TestPoint
- added TP261: GCL, TestPoint:TestPoint_Pad_D1.5mm, symbol Connector:TestPoint
- added TP262: SOURCE_C, TestPoint:TestPoint_Pad_D1.5mm, symbol Connector:TestPoint
Connections:
- net GAH: now also TP220.1
- net GAL: now also TP221.1
- net GBH: now also TP240.1
- net GBL: now also TP241.1
- net GCH: now also TP260.1
- net GCL: now also TP261.1
- net SOURCE_A: now also TP222.1
- net SOURCE_B: now also TP242.1
- net SOURCE_C: now also TP262.1
Other:
- note added: "Main CSA: 1.5 V zero, 20 mV/A Gate probes need local source returns. High-side VGS: differential probe only."
- note removed: "Main CSA: 1.5 V zero, 20 mV/A DRV CSA: diagnostic channel"
- moved on the sheet: C210, C211, C212, C213, C214, C215, C230, C231, C232, C233, C234, C235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

Commit message: devlog 04
Parts:
- C210, C211, C230, C231, C250, C251: Manufacturer (none) -> TDK
- C212, C232, C252: MPN GRM188R71H104KA93D -> C0603C104K5RACTU; Manufacturer Murata -> KEMET
- C213, C214, C215, C233, C234, C235, C253, C254, C255: Manufacturer (none) -> KEMET
- U202, U203, U204: value INA241A2DR -> INA241A2IDR; MPN INA241A2DR -> INA241A2IDR
Connections:
- net VBIAS_1V5 renamed VBIAS_1V25
Other:
- note added: "Main CSA: 1.25 V zero, 20 mV/A Gate probes need local source returns. High-side VGS: differential probe only."
- note removed: "Main CSA: 1.5 V zero, 20 mV/A Gate probes need local source returns. High-side VGS: differential probe only."

Commit message: connect the bridge test points and snubbers
Parts:
- TP220, TP221, TP222, TP240, TP241, TP242, TP260, TP261, TP262: footprint TestPoint:TestPoint_Pad_D1.5mm -> bldc-esc:TestPoint_Pad_D1.5mm_NoSilk
Changed lines of the file:
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@@
       )
     )
-    (property "Footprint" "TestPoint:TestPoint_Pad_D1.5mm"
+    (property "Footprint" "bldc-esc:TestPoint_Pad_D1.5mm_NoSilk"
       (at 50.8 54.61 0)
       (effects
@@
       )
     )
-    (property "Footprint" "TestPoint:TestPoint_Pad_D1.5mm"
+    (property "Footprint" "bldc-esc:TestPoint_Pad_D1.5mm_NoSilk"
       (at 50.8 90.17 0)
       (effects
@@
       )
     )
-    (property "Footprint" "TestPoint:TestPoint_Pad_D1.5mm"
+    (property "Footprint" "bldc-esc:TestPoint_Pad_D1.5mm_NoSilk"
       (at 91.44 118.11 0)
       (effects
@@
       )
     )
-    (property "Footprint" "TestPoint:TestPoint_Pad_D1.5mm"
+    (property "Footprint" "bldc-esc:TestPoint_Pad_D1.5mm_NoSilk"
       (at 176.53 54.61 0)
       (effects
@@
       )
     )
-    (property "Footprint" "TestPoint:TestPoint_Pad_D1.5mm"
+    (property "Footprint" "bldc-esc:TestPoint_Pad_D1.5mm_NoSilk"
       (at 176.53 90.17 0)
       (effects
@@
       )
     )
-    (property "Footprint" "TestPoint:TestPoint_Pad_D1.5mm"
+    (property "Footprint" "bldc-esc:TestPoint_Pad_D1.5mm_NoSilk"
       (at 217.17 118.11 0)
       (effects
@@
       )
     )
-    (property "Footprint" "TestPoint:TestPoint_Pad_D1.5mm"
+    (property "Footprint" "bldc-esc:TestPoint_Pad_D1.5mm_NoSilk"
       (at 302.26 54.61 0)
       (effects
@@
       )
     )
-    (property "Footprint" "TestPoint:TestPoint_Pad_D1.5mm"
+    (property "Footprint" "bldc-esc:TestPoint_Pad_D1.5mm_NoSilk"
       (at 302.26 90.17 0)
       (effects
@@
       )
     )
-    (property "Footprint" "TestPoint:TestPoint_Pad_D1.5mm"
+    (property "Footprint" "bldc-esc:TestPoint_Pad_D1.5mm_NoSilk"
       (at 342.9 118.11 0)
       (effects
