File: schematic/01_dc_link.kicad_sch (KiCad schematic)
At the start: 0 parts

Commit message: devlog 02
Parts:
- added C101, C102, C103, C104, C105, C106, C107, C108, C115, C116: 100u 63V, Capacitor_SMD:CP_Elec_10x12.5, symbol Device:C_Polarized
- added C109: 4.7n 1kV, Capacitor_SMD:C_1206_3216Metric, symbol Device:C
- added D101: SMCJ30A, Diode_SMD:D_SMC, symbol Device:D_TVS
- added J101: XT60PW-M, Connector_AMASS:AMASS_XT60PW-M_1x02_P7.20mm_Horizontal, symbol Connector_Generic:Conn_01x02
- added J102: MT60 / 12AWG pigtail, bldc-esc:MT60_Pigtail_12AWG, symbol Connector_Generic:Conn_01x03
- added J103: CHASSIS, Connector_PinHeader_2.54mm:PinHeader_1x02_P2.54mm_Vertical, symbol Connector_Generic:Conn_01x02
- added R101: 10k, Resistor_SMD:R_1206_3216Metric, symbol Device:R
- added R102: 1M, Resistor_SMD:R_0603_1608Metric, symbol Device:R
- added R103: 0, Resistor_SMD:R_0603_1608Metric, symbol Device:R
- added TP101: VBUS, TestPoint:TestPoint_Pad_D1.5mm, symbol Connector:TestPoint
- added TP102: GND, TestPoint:TestPoint_Pad_D1.5mm, symbol Connector:TestPoint
- added TP103: PHASE_A, TestPoint:TestPoint_Pad_D1.5mm, symbol Connector:TestPoint
- added TP104: PHASE_B, TestPoint:TestPoint_Pad_D1.5mm, symbol Connector:TestPoint
- added TP105: PHASE_C, TestPoint:TestPoint_Pad_D1.5mm, symbol Connector:TestPoint
Connections:
- new net CHASSIS: C109.1, J103.1 (Pin_1), R102.1, R103.1
- new net GND: C101.1, C101.2, C102.1, C102.2, C103.1, C103.2, C104.1, C104.2, C105.1, C105.2, C106.1, C106.2, C107.1, C107.2, C108.1, C108.2, C109.2, C115.1, C115.2, C116.1, C116.2, D101.1 (A1), D101.2 (A2), J101.1 (Pin_1), J101.2 (Pin_2), J103.2 (Pin_2), R101.1, R101.2, R102.2, R103.2, TP101.1, TP102.1
- new net PHASE_A: J102.1 (Pin_1), TP103.1
- new net PHASE_B: J102.2 (Pin_2), TP104.1
- new net PHASE_C: J102.3 (Pin_3), TP105.1
Other:
- note added: "12-30 V operating bus. External DC-rated fuse required close to the source. No electronic reverse-polarity protection."
- note added: "C101-C108, C115-C116: 10 x 100 uF / 63 V hybrid, 1,000 uF total. Bulk bank does not absorb sustained regeneration."
- note added: "DC input and local energy storage"
- note added: "DC input and motor connections"
- note added: "MT60 pigtail: 1=A, 2=B, 3=C. Provide strain relief."
- note added: "Motor cable / test points"
- note added: "R103 is DNP. Select the chassis bond after enclosure and EMI review."
- note added: "Shield / chassis connection"
- title: (none) -> DC input and motor connections

Commit message: devlog 03
Other:
- moved on the sheet: C101, C102, C103, C104, C105, C106, C107, C108, C115, C116, D101, J102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

Commit message: devlog 04
Parts:
- C109: MPN C1206C472KGRACTU -> C1206C472KDRACTU; Manufacturer (none) -> KEMET
- D101: symbol Device:D_TVS -> Device:D_Zener; Manufacturer (none) -> Littelfuse
- J101, J102: Manufacturer (none) -> AMASS
- J103: Manufacturer (none) -> Harwin
Other:
- moved on the sheet: C101, C102, C103, C104, C105, C106, C107, C108, C109, C115, C116, D101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

Commit message: connect the bridge test points and snubbers
Parts:
- TP103, TP104, TP105: footprint TestPoint:TestPoint_Pad_D1.5mm -> bldc-esc:TestPoint_Pad_D1.5mm_NoSilk
Changed lines of the file:
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@@
       )
     )
-    (property "Footprint" "TestPoint:TestPoint_Pad_D1.5mm"
+    (property "Footprint" "bldc-esc:TestPoint_Pad_D1.5mm_NoSilk"
       (at 133.35 152.4 0)
       (effects
@@
       )
     )
-    (property "Footprint" "TestPoint:TestPoint_Pad_D1.5mm"
+    (property "Footprint" "bldc-esc:TestPoint_Pad_D1.5mm_NoSilk"
       (at 149.86 152.4 0)
       (effects
@@
       )
     )
-    (property "Footprint" "TestPoint:TestPoint_Pad_D1.5mm"
+    (property "Footprint" "bldc-esc:TestPoint_Pad_D1.5mm_NoSilk"
       (at 166.37 152.4 0)
       (effects

Commit message: add mounting holes and bring-up firmware
Parts:
- J101: footprint Connector_AMASS:AMASS_XT60PW-M_1x02_P7.20mm_Horizontal -> bldc-esc:XT60PW_M_Edge
Changed lines of the file:
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@@
       )
     )
-    (property "Footprint" "Connector_AMASS:AMASS_XT60PW-M_1x02_P7.20mm_Horizontal"
+    (property "Footprint" "bldc-esc:XT60PW_M_Edge"
       (at 16.51 59.69 0)
       (effects
