File: schematic/03_regen.kicad_sch (KiCad schematic)
At the start: 44 parts, among them J301 DUMP RESISTOR, Q301 ISC011N06LM5, Q302 2N7002, U301 TLV3011BDBVR, U302 UCC27511ADBVR, U303 INA180A1IDBVR, U304 TLV3201AIDBVR, U305 TPS3808G50DBVR, U306 SN74LVC1G17DBVR, U307 SN74LVC1G74DCTR

Commit message: devlog 03
Parts:
- removed C307, C309, C311: 100n 50V, Capacitor_SMD:C_0603_1608Metric, symbol Device:C
- removed C308: 100p 50V, Capacitor_SMD:C_0603_1608Metric, symbol Device:C
- removed C310: 10n 50V, Capacitor_SMD:C_0603_1608Metric, symbol Device:C
- removed D302, D303: BAT54H, Diode_SMD:D_SOD-123F, symbol Device:D
- removed R311, R312, R313: 10k, Resistor_SMD:R_0603_1608Metric, symbol Device:R
- removed R314, R315, R316, R317, R318: 100k, Resistor_SMD:R_0603_1608Metric, symbol Device:R
- removed U304: TLV3201AIDBVR, Package_TO_SOT_SMD:SOT-23-5, symbol bldc-esc:TLV3201
- removed U305: TPS3808G50DBVR, Package_TO_SOT_SMD:SOT-23-6, symbol bldc-esc:TPS3808Gxx
- removed U306: SN74LVC1G17DBVR, Package_TO_SOT_SMD:SOT-23-5, symbol 74xGxx:74LVC1G17
- removed U307: SN74LVC1G74DCTR, Package_SO:SSOP-8_2.95x2.8mm_P0.65mm, symbol bldc-esc:SN74LVC1G74
- added C313: 100n 50V, Capacitor_SMD:C_0603_1608Metric, symbol Device:C
- added C314: 1u 16V, Capacitor_SMD:C_0603_1608Metric, symbol Device:C
- added U308: REF2025AIDDCR, Package_TO_SOT_SMD:SOT-23-5, symbol Reference_Voltage:REF2025
- C303: value 1n 50V -> 100n 50V; MPN C0603C102J5GACTU -> GRM188R71H104KA93D; Manufacturer (none) -> Murata
- D301: value STPS5H100B -> STPS5H100AF; footprint Diode_SMD:D_SMC -> Diode_SMD:D_SOD-128; symbol Device:D -> Device:D_Schottky; MPN STPS5H100B -> STPS5H100AF; Manufacturer (none) -> STMicroelectronics
Connections:
- net 5V_BUS: now also C313.1, U308.3 (EN), U308.4 (IN)
- net DUMP_REF: now also U308.1 (Vbias); no longer U301.5 (REF)
- net GND: now also C313.2, C314.2, U308.2 (GND)
- new net DUMP_REF_2V5: C314.1, U308.5 (Vref)
Other:
- note added: "External dump resistor: 2-25 ohm; pulse/thermal rating required. Chopper trip: about 20.8 A, power-cycle reset. Reference U308 stays bus-powered."
- note added: "Independent bus clamp / nominal 31.3 V on, 30.6 V off"
- note removed: "5 V-to-3.3 V monitor dividers"
- note removed: "Chopper overcurrent trip and power-cycle latch"
- note removed: "External dump resistor: 2-25 ohm; pulse/thermal rating required. Chopper trip: about 20.7 A, power-cycle reset."
- note removed: "Independent bus clamp / nominal 31.0 V on, 30.5 V off"
- moved on the sheet: C301, C302, C303, C304, C305, C306, D301, J301, Q301, Q302, R301, R302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

Commit message: devlog 04
Parts:
- C301: Manufacturer (none) -> KEMET
- C302, C303, C304, C306, C313: MPN GRM188R71H104KA93D -> C0603C104K5RACTU; Manufacturer Murata -> KEMET
- C305, C314: MPN GRM188R71C105KA12D -> C0603C105K4RACTU; Manufacturer (none) -> KEMET
- J301: Manufacturer (none) -> Phoenix Contact
- U301: value TLV3011BDBVR -> TLV3011BIDBVR; MPN TLV3011BDBVR -> TLV3011BIDBVR
Other:
- moved on the sheet: C306, D301, J301, TP301, U303

Commit message: fix part order codes and record supplier quotes
Parts:
- R310: MPN WSLP2512R0030FEA -> WSLP25123L000FEA
Changed lines of the file:
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@@
       (hide yes)
     )
-    (property "MPN" "WSLP2512R0030FEA"
+    (property "MPN" "WSLP25123L000FEA"
       (at 278.13 128.27 0)
       (effects
