File: schematic/07_io_can.kicad_sch (KiCad schematic)
At the start: 0 parts

Commit message: devlog 02
Parts:
- added C704: 100n 50V, Capacitor_SMD:C_0603_1608Metric, symbol Device:C
- added D703: PESD2CANFD24V-T, Package_TO_SOT_SMD:SOT-23, symbol bldc-esc:PESD2CANFD24V_T
- added J701: CAN, Connector_JST:JST_GH_BM03B-GHS-TBT_1x03-1MP_P1.25mm_Vertical, symbol Connector_Generic:Conn_01x03
- added J702: UART / 3V3, Connector_JST:JST_GH_BM04B-GHS-TBT_1x04-1MP_P1.25mm_Vertical, symbol Connector_Generic:Conn_01x04
- added JP701: CAN TERM, Connector_PinHeader_2.54mm:PinHeader_1x02_P2.54mm_Vertical, symbol Connector_Generic:Conn_01x02
- added R717, R718: 10k, Resistor_SMD:R_0603_1608Metric, symbol Device:R
- added R719: 120, Resistor_SMD:R_0805_2012Metric, symbol Device:R
- added U709: TCAN3403DRQ1, Package_SO:SOIC-8_3.9x4.9mm_P1.27mm, symbol bldc-esc:TCAN3403
Connections:
- new net 3V3: C704.1, J702.4 (Pin_4), R717.1, R718.1, U709.3 (VCC), U709.5 (VIO)
- new net CAN_H: D703.1 (CANH), J701.2 (Pin_2), R719.1, U709.7 (CANH)
- new net CAN_L: D703.2 (CANL), J701.3 (Pin_3), JP701.2 (Pin_2), U709.6 (CANL)
- new net CAN_RX: U709.4 (RXD)
- new net CAN_STB: R717.2, U709.8 (STB)
- new net CAN_TERM: JP701.1 (Pin_1), R719.2
- new net CAN_TX: R718.2, U709.1 (TXD)
- new net GND: C704.2, D703.3 (GND), J701.1 (Pin_1), J702.1 (Pin_1), U709.2 (GND)
- new net UART_RX: J702.3 (Pin_3)
- new net UART_TX: J702.2 (Pin_2)
Other:
- note added: "CAN FD"
- note added: "CAN FD and UART"
- note added: "JP701 fitted = 120 ohm termination. Fit termination only at the two ends of the CAN bus."
- note added: "TX and RX are named from the controller. Not an RS-232 or 5 V serial port."
- note added: "UART / 3.3 V logic"
- title: (none) -> CAN FD and UART

Commit message: devlog 03
Parts:
- added C706: 1u 16V, Capacitor_SMD:C_0603_1608Metric, symbol Device:C
Connections:
- net 3V3: now also C706.1
- net GND: now also C706.2
Other:
- note added: "Short local 3.3 V wiring only; TX/RX are controller-side names. Not an RS-232 or 5 V port. Supply pin is an output, not a power input."
- note removed: "TX and RX are named from the controller. Not an RS-232 or 5 V serial port."
- moved on the sheet: D703, J701, J702, JP701, R719

Commit message: devlog 04
Parts:
- C704: MPN GRM188R71H104KA93D -> C0603C104K5RACTU; Manufacturer Murata -> KEMET
- C706: MPN GRM188R71C105KA12D -> C0603C105K4RACTU; Manufacturer (none) -> KEMET
- JP701: Manufacturer (none) -> Harwin
Other:
- moved on the sheet: J702
Changed lines of the file:
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@@
   )
   (text "Short local 3.3 V wiring only; TX/RX are controller-side names.\nNot an RS-232 or 5 V port. Supply pin is an output, not a power input."
-    (at 125.73 158.75 0)
+    (at 123.19 158.75 0)
     (effects
       (font
@@
       (hide yes)
     )
-    (property "MPN" "GRM188R71H104KA93D"
+    (property "MPN" "C0603C104K5RACTU"
       (at 35.56 48.26 0)
       (effects
@@
       (hide yes)
     )
-    (property "Manufacturer" "Murata"
+    (property "Manufacturer" "KEMET"
       (at 35.56 48.26 0)
       (effects
@@
       (hide yes)
     )
-    (property "MPN" "GRM188R71C105KA12D"
+    (property "MPN" "C0603C105K4RACTU"
       (at 62.23 48.26 0)
       (effects
@@
       (hide yes)
     )
-    (property "Manufacturer" ""
+    (property "Manufacturer" "KEMET"
       (at 62.23 48.26 0)
       (effects
@@
       (hide yes)
     )
-    (property "Manufacturer" ""
+    (property "Manufacturer" "Harwin"
       (at 179.07 128.27 0)
       (effects
@@
   (symbol
     (lib_id "Connector_Generic:Conn_01x04")
-    (at 49.53 158.75 0)
+    (at 46.99 158.75 0)
     (unit 1)
     (exclude_from_sim no)
@@
     (dnp no)
     (property "Reference" "J702"
-      (at 53.34 156.21 0)
+      (at 50.8 156.21 0)
       (effects
         (font
@@
     )
     (property "Value" "UART / 3V3"
-      (at 53.34 158.75 0)
+      (at 50.8 158.75 0)
       (effects
         (font
@@
     )
     (property "Footprint" "Connector_JST:JST_GH_BM04B-GHS-TBT_1x04-1MP_P1.25mm_Vertical"
-      (at 49.53 158.75 0)
+      (at 46.99 158.75 0)
       (effects
         (font
@@
     )
     (property "Datasheet" ""
-      (at 49.53 158.75 0)
+      (at 46.99 158.75 0)
       (effects
         (font
@@
     )
     (property "MPN" "BM04B-GHS-TBT(LF)(SN)"
-      (at 49.53 158.75 0)
+      (at 46.99 158.75 0)
       (effects
         (font
@@
     )
     (property "Manufacturer" "JST"
-      (at 49.53 158.75 0)
+      (at 46.99 158.75 0)
       (effects
         (font
@@
   )
   (symbol
-    (lib_id "power:GND")
-    (at 184.15 69.85 0)
-    (unit 1)
-    (exclude_from_sim no)
-    (in_bom no)
-    (on_board yes)
-    (dnp no)
-    (property "Reference" "#PWR070003"
-      (at 184.15 69.85 0)
-      (effects
-        (font
-          (size 1.0 1.0)
-        )
-        (hide yes)
-      )
-    )
-    (property "Value" "GND"
-      (at 184.15 73.66 0)
-      (effects
-        (font
-          (size 1.0 1.0)
-        )
-      )
-    )
-    (instances
-      (project "bldc-esc"
-        (path "/10000000-0000-4000-8000-000000000000/10000000-0000-4000-8000-000000000007"
-          (reference "#PWR070003")
-          (unit 1)
-        )
-      )
-    )
-  )
-  (symbol
-    (lib_id "power:GND")
-    (at 24.13 156.21 0)
-    (unit 1)
-    (exclude_from_sim no)
-    (in_bom no)
-    (on_board yes)
-    (dnp no)
-    (property "Reference" "#PWR070004"
-      (at 24.13 156.21 0)
-      (effects
-        (font
-          (size 1.0 1.0)
-        )
-        (hide yes)
-      )
-    )
-    (property "Value" "GND"
-      (at 24.13 160.02 0)
-      (effects
-        (font
-          (size 1.0 1.0)
-        )
-      )
-    )
-    (instances
-      (project "bldc-esc"
-        (path "/10000000-0000-4000-8000-000000000000/10000000-0000-4000-8000-000000000007"
-          (reference "#PWR070004")
-          (unit 1)
-        )
-      )
-    )
-  )
-  (symbol
     (lib_id "power:VCC")
     (at 16.51 163.83 0)
@@
     (on_board yes)
     (dnp no)
-    (property "Reference" "#PWR070005"
+    (property "Reference" "#PWR070003"
       (at 16.51 163.83 0)
       (effects
@@
       (project "bldc-esc"
         (path "/10000000-0000-4000-8000-000000000000/10000000-0000-4000-8000-000000000007"
-          (reference "#PWR070005")
+          (reference "#PWR070003")
           (unit 1)
         )
@@
     (on_board yes)
     (dnp no)
-    (property "Reference" "#PWR070006"
+    (property "Reference" "#PWR070004"
       (at 57.15 73.66 0)
       (effects
@@
       (project "bldc-esc"
         (path "/10000000-0000-4000-8000-000000000000/10000000-0000-4000-8000-000000000007"
-          (reference "#PWR070006")
+          (reference "#PWR070004")
           (unit 1)
         )
@@
     (on_board yes)
     (dnp no)
-    (property "Reference" "#PWR070007"
+    (property "Reference" "#PWR070005"
       (at 99.06 86.36 0)
       (effects
@@
       (project "bldc-esc"
         (path "/10000000-0000-4000-8000-000000000000/10000000-0000-4000-8000-000000000007"
-          (reference "#PWR070007")
+          (reference "#PWR070005")
           (unit 1)
         )
@@
     (on_board yes)
     (dnp no)
-    (property "Reference" "#PWR070008"
+    (property "Reference" "#PWR070006"
       (at 35.56 39.37 0)
       (effects
@@
       (project "bldc-esc"
         (path "/10000000-0000-4000-8000-000000000000/10000000-0000-4000-8000-000000000007"
-          (reference "#PWR070008")
+          (reference "#PWR070006")
           (unit 1)
         )
@@
     (on_board yes)
     (dnp no)
-    (property "Reference" "#PWR070009"
+    (property "Reference" "#PWR070007"
       (at 35.56 57.15 0)
       (effects
@@
       (project "bldc-esc"
         (path "/10000000-0000-4000-8000-000000000000/10000000-0000-4000-8000-000000000007"
-          (reference "#PWR070009")
+          (reference "#PWR070007")
           (unit 1)
         )
@@
     (on_board yes)
     (dnp no)
-    (property "Reference" "#PWR070010"
+    (property "Reference" "#PWR070008"
       (at 16.51 73.66 0)
       (effects
@@
       (project "bldc-esc"
         (path "/10000000-0000-4000-8000-000000000000/10000000-0000-4000-8000-000000000007"
-          (reference "#PWR070010")
+          (reference "#PWR070008")
           (unit 1)
         )
@@
     (on_board yes)
     (dnp no)
-    (property "Reference" "#PWR070011"
+    (property "Reference" "#PWR070009"
       (at 16.51 106.68 0)
       (effects
@@
       (project "bldc-esc"
         (path "/10000000-0000-4000-8000-000000000000/10000000-0000-4000-8000-000000000007"
-          (reference "#PWR070011")
+          (reference "#PWR070009")
           (unit 1)
         )
@@
     (on_board yes)
     (dnp no)
-    (property "Reference" "#PWR070012"
+    (property "Reference" "#PWR070010"
       (at 148.59 116.84 0)
       (effects
@@
       (project "bldc-esc"
         (path "/10000000-0000-4000-8000-000000000000/10000000-0000-4000-8000-000000000007"
-          (reference "#PWR070012")
+          (reference "#PWR070010")
           (unit 1)
         )
@@
     (pts
       (xy 16.51 163.83)
-      (xy 44.45 163.83)
+      (xy 41.91 163.83)
     )
     (stroke
@@
     (pts
       (xy 24.13 156.21)
-      (xy 44.45 156.21)
+      (xy 41.91 156.21)
     )
     (stroke
@@
   (wire
     (pts
-      (xy 39.37 161.29)
-      (xy 44.45 161.29)
-    )
-    (stroke
-      (width 0)
-      (type default)
-    )
-  )
-  (wire
-    (pts
-      (xy 39.37 158.75)
-      (xy 44.45 158.75)
+      (xy 36.83 161.29)
+      (xy 41.91 161.29)
+    )
+    (stroke
+      (width 0)
+      (type default)
+    )
+  )
+  (wire
+    (pts
+      (xy 36.83 158.75)
+      (xy 41.91 158.75)
     )
     (stroke
@@
     (diameter 0)
     (color 0 0 0 0)
+  )
+  (global_label "GND"
+    (shape bidirectional)
+    (at 184.15 69.85 180)
+    (effects
+      (font
+        (size 0.95 0.95)
+      )
+      (justify right)
+    )
   )
   (label "CAN_TERM"
@@
     )
   )
+  (global_label "GND"
+    (shape bidirectional)
+    (at 24.13 156.21 180)
+    (effects
+      (font
+        (size 0.95 0.95)
+      )
+      (justify right)
+    )
+  )
   (global_label "CAN_RX"
     (shape bidirectional)
@@
   (global_label "UART_TX"
     (shape bidirectional)
-    (at 39.37 158.75 180)
+    (at 36.83 158.75 180)
     (effects
       (font
@@
   (global_label "UART_RX"
     (shape bidirectional)
-    (at 39.37 161.29 180)
+    (at 36.83 161.29 180)
     (effects
       (font

Commit message: fix part order codes and record supplier quotes
Parts:
- D703: MPN PESD2CANFD24V-T,215 -> PESD2CANFD24V-TR
Changed lines of the file:
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@@
       (hide yes)
     )
-    (property "MPN" "PESD2CANFD24V-T,215"
+    (property "MPN" "PESD2CANFD24V-TR"
       (at 132.08 118.11 0)
       (effects
